Commit message: robot control integration with gazebo done

File: differential_robot_description/urdf/common_properties.xacro (robot description, xacro)
@@ -10,4 +10,7 @@
     <material name="gray">
         <color rgba="0.5 0.5 0.5 1.0"/>
+    </material>
+    <material name="red_collision">
+        <color rgba="0.5 0.0 0.0 0.5"/>
     </material>
     <!-- Inertial macros -->

File: differential_robot_description/urdf/differential_robot.urdf.xacro (robot description, xacro)
@@ -3,3 +3,4 @@
     <xacro:include filename="$(find differential_robot_description)/urdf/common_properties.xacro"/>
     <xacro:include filename="$(find differential_robot_description)/urdf/mobile_base.xacro"/>
+    <xacro:include filename="$(find differential_robot_description)/urdf/mobile_base_gazebo.xacro"/>
 </robot>

File: differential_robot_description/urdf/mobile_base.xacro (robot description, xacro)
@@ -8,5 +8,5 @@
     <xacro:macro name="wheel_link" params="prefix">
         <link name="${prefix}_wheel_link">
-            <xacro:cylinder_inertia m="1.0" r="${wheel_radius}" l="${wheel_lenght}" xyz="0.0 0.0 0.0" rpy="${pi/2.0} 0.0 0.0"/>
+            <xacro:cylinder_inertia m="1.0" r="${2*wheel_radius}" l="${2*wheel_lenght}" xyz="0.0 0.0 0.0" rpy="${pi/2.0} 0.0 0.0"/>
             <visual>
                 <geometry>
@@ -17,5 +17,9 @@
             </visual>
             <collision>
-                <origin xyz="0.0 0.0 0.0" rpy="0.0 0.0 0.0"/>
+                <geometry>
+                    <cylinder radius="${wheel_radius}" length="${wheel_lenght}"/>
+                </geometry>
+                <origin xyz="0.0 0.0 0.0" rpy="${pi/2.0} 0.0 0.0"/>
+                <!-- <material name="red_collison"/> -->
             </collision>
         </link>
@@ -24,5 +28,5 @@
     <link name="base_footprint"/>
     <link name="base_link">
-        <xacro:box_inertia m="5.0" l="${base_lenght}" w="${base_width}" h="${base_height}"
+        <xacro:box_inertia m="5.0" l="${2*base_lenght}" w="${2*base_width}" h="${2*base_height}"
                            xyz="0.0 0.0 ${base_height/2.0}" rpy="0.0 0.0 0.0"/>
         <visual>
@@ -34,5 +38,9 @@
         </visual>
         <collision>
-            <origin xyz="0.0 0.0 0.0" rpy="0.0 0.0 0.0"/>
+            <geometry>
+                <box size="${base_lenght} ${base_width} ${base_height}"/>
+            </geometry>
+            <origin xyz="0.0 0.0 ${base_height/2.0}" rpy="0.0 0.0 0.0"/>
+            <!-- <material name="red_collison"/> -->
         </collision>
     </link>
@@ -58,5 +66,5 @@
     </link> -->
     <link name="caster_wheel_link">
-        <xacro:sphere_inertia m="0.5" r="${wheel_radius/2.0}"
+        <xacro:sphere_inertia m="0.5" r="${2*wheel_radius/2.0}"
                            xyz="0.0 0.0 0.0" rpy="0.0 0.0 0.0"/>
         <visual>
@@ -68,5 +76,9 @@
         </visual>
         <collision>
+            <geometry>
+                <sphere radius="${wheel_radius/2.0}"/>
+            </geometry>
             <origin xyz="0.0 0.0 0.0" rpy="0.0 0.0 0.0"/>
+            <!-- <material name="red_collison"/> -->
         </collision>
     </link>
