Commit message: Added a lidar, still doesnt work

File: differential_robot_description/urdf/camera.xacro (robot description, xacro)
@@ -6,5 +6,4 @@
     <link name="camera_link">
         <visual>
-            <xacro:box_inertia m="0.1" l="${camera_lenght}" w="${camera_width}" h="${camera_height}" xyz="0.0 0.0 0.0" rpy="0.0 0.0 0.0"/>
             <geometry>
                 <box size="${camera_lenght} ${camera_width} ${camera_height}"/>
@@ -12,11 +11,12 @@
             <origin xyz="0.0 0.0 0.0" rpy="0.0 0.0 0.0"/>
             <material name="blue"/>
-            <collision>
-                <geometry>
-                    <box size="${camera_lenght} ${camera_width} ${camera_height}"/>
-                </geometry>
-                <origin xyz="0.0 0.0 0.0" rpy="0.0 0.0 0.0"/>
-            </collision>
         </visual>
+        <collision>
+            <geometry>
+                <box size="${camera_lenght} ${camera_width} ${camera_height}"/>
+            </geometry>
+            <origin xyz="0.0 0.0 0.0" rpy="0.0 0.0 0.0"/>
+        </collision>
+        <xacro:box_inertia m="0.1" l="${camera_lenght}" w="${camera_width}" h="${camera_height}" xyz="0.0 0.0 0.0" rpy="0.0 0.0 0.0"/>
     </link>
     <!-- generate an optical frame

File: differential_robot_description/urdf/common_properties.xacro (robot description, xacro)
@@ -13,4 +13,7 @@
     <material name="red_collision">
         <color rgba="0.5 0.0 0.0 0.5"/>
+    </material>
+    <material name="black">
+        <color rgba="0.0 0.0 0.0 1.0"/>
     </material>
     <!-- Inertial macros -->

File: differential_robot_description/urdf/differential_robot.urdf.xacro (robot description, xacro)
@@ -5,3 +5,4 @@
     <xacro:include filename="$(find differential_robot_description)/urdf/mobile_base_gazebo.xacro"/>
     <xacro:include filename="$(find differential_robot_description)/urdf/camera.xacro"/>
+    <xacro:include filename="$(find differential_robot_description)/urdf/lidar.xacro"/>
 </robot>
