Commit message: lidar corrected

File: differential_robot_description/urdf/lidar.xacro (robot description, xacro)
@@ -24,5 +24,5 @@
         <child link="lidar_link"/>
         <axis xyz="0 0 1" />
-        <origin xyz="0 0 ${base_height}" rpy="0 0 0"/>
+        <origin xyz="0 0 ${base_height + lidar_lenght / 2.0}" rpy="0 0 0"/>
     </joint>
     <gazebo reference="lidar_link">
@@ -30,5 +30,5 @@
         <sensor type="ray" name="lidar_sensor">
             <pose>0 0 0 0 0 0</pose>
-            <visualize>false</visualize>
+            <visualize>true</visualize>
             <update_rate>40</update_rate>
             <ray>

Commit message: Solved the laser scan problem, lidar works now

File: differential_robot_description/urdf/lidar.xacro (robot description, xacro)
@@ -2,5 +2,5 @@
 <robot xmlns:xacro="http://www.ros.org/wiki/xacro">
     <xacro:property name="lidar_radius" value="0.05"/>
-    <xacro:property name="lidar_lenght" value="0.1"/>
+    <xacro:property name="lidar_lenght" value="0.05"/>
     <!-- Hokuyo Laser -->
     <link name="lidar_link">
@@ -14,5 +14,5 @@
         <collision>
             <geometry>
-                <box size="0.1 0.1 0.1"/>
+                <cylinder radius="${lidar_radius}" length="${lidar_lenght}"/>
             </geometry>
             <origin xyz="0 0 0" rpy="0 0 0"/>
@@ -29,4 +29,5 @@
         <material>Gazebo/Black</material>
         <sensor type="ray" name="lidar_sensor">
+            <always_on>true</always_on>
             <pose>0 0 0 0 0 0</pose>
             <visualize>true</visualize>
@@ -34,28 +35,34 @@
             <ray>
                 <scan>
-                <horizontal>
-                    <samples>720</samples>
-                    <resolution>1</resolution>
-                    <min_angle>-1.570796</min_angle>
-                    <max_angle>1.570796</max_angle>
-                </horizontal>
+                    <horizontal>
+                        <samples>720</samples>
+                        <resolution>1</resolution>
+                        <!-- <min_angle>-1.570796</min_angle>
+                        <max_angle>1.570796</max_angle> -->
+                        <min_angle>-2.094395</min_angle>
+                        <max_angle>2.094395</max_angle>
+                    </horizontal>
                 </scan>
                 <range>
-                <min>0.10</min>
-                <max>30.0</max>
-                <resolution>0.01</resolution>
+                    <min>0.10</min>
+                    <max>30.0</max>
+                    <resolution>0.01</resolution>
                 </range>
                 <noise>
-                <type>gaussian</type>
-                <!-- Noise parameters based on published spec for Hokuyo laser
-                    achieving "+-30mm" accuracy at range < 10m.  A mean of 0.0m and
-                    stddev of 0.01m will put 99.7% of samples within 0.03m of the true
-                    reading. -->
-                <mean>0.0</mean>
-                <stddev>0.01</stddev>
+                    <type>gaussian</type>
+                    <!-- Noise parameters based on published spec for Hokuyo laser
+                        achieving "+-30mm" accuracy at range < 10m.  A mean of 0.0m and
+                        stddev of 0.01m will put 99.7% of samples within 0.03m of the true
+                        reading. -->
+                    <mean>0.0</mean>
+                    <stddev>0.01</stddev>
                 </noise>
             </ray>
-            <plugin name="gazebo_ros_head_hokuyo_controller" filename="libgazebo_ros_laser.so">
-                <topicName>/scan</topicName>
+            <plugin name="gazebo_ros_lidar_controller" filename="libgazebo_ros_ray_sensor.so">
+                <ros>
+                    <!-- <namespace>lidar</namespace> -->
+                    <remapping>~/out:=scan</remapping>
+                </ros>
+                <output_type>sensor_msgs/LaserScan</output_type>
                 <frameName>lidar_link</frameName>
             </plugin>
