Commit message: In process of making the gripper static

File: custom_robotiq_description/urdf/robotiq_2f85_gripper.urdf.xacro (robot description, xacro)
@@ -2,8 +2,11 @@
 <robot xmlns:xacro="http://www.ros.org/wiki/xacro" name="robotiq_gripper">
     <!-- parameters -->
+    <xacro:arg name="prefix" default="" />
     <xacro:arg name="bringup" default="true" />
     <!-- Import macros -->
     <xacro:include filename="$(find custom_robotiq_description)/urdf/robotiq_2f85_macro.urdf.xacro" />
+    <xacro:include filename="$(find custom_robotiq_description)/urdf/robotiq_camera.xacro" />
     <link name="world" />
-    <xacro:robotiq_gripper name="RobotiqGripperHardwareInterface" prefix="" parent="world" bringup="$(arg bringup)"/>
+    <xacro:robotiq_camera prefix="$(arg prefix)" parent="world"/>
+    <xacro:robotiq_gripper name="RobotiqGripperHardwareInterface" prefix="$(arg prefix)" parent="robotiq_camera" bringup="$(arg bringup)" fixed="true"/>
 </robot>

File: custom_robotiq_description/urdf/robotiq_2f85_macro.urdf.xacro (robot description, xacro)
@@ -5,5 +5,6 @@
         prefix
         parent
-        bringup:=false">
+        bringup:=false
+        fixed:=true">
         <xacro:unless value="${bringup}">
             <!-- Robotiq 2f-85 TRANSMISSION -->
@@ -12,34 +13,4 @@
         </xacro:unless>
         <!-- Robotiq camera -->
-        <link name="${prefix}robotiq_camera">
-            <visual>
-                <geometry>
-                    <mesh filename="file://$(find custom_robotiq_description)/meshes/robotiq_wrist_camera.stl" scale="0.001 0.001 0.001"/>
-                </geometry>
-                <origin xyz="-37.875e-03 -37.875e-03 -6.5e-03" rpy="0 0 0" />
-            </visual>
-            <collision>
-                <geometry>
-                    <mesh filename="file://$(find custom_robotiq_description)/meshes/robotiq_wrist_camera.stl" scale="0.001 0.001 0.001"/>
-                </geometry>
-                <origin xyz="-37.875e-03 -37.875e-03 -6.5e-03" rpy="0 0 0" />
-            </collision>
-            <inertial>
-                <origin xyz="-6.5e-03 6.6e-03 4.0e-03" rpy="0 0 0" />
-                <mass value="0.195" />
-                <inertia ixx="6.69695624e-05" ixy="5.21511788e-09" ixz="-2.74383009e-08"
-                        iyy="7.85088161e-05" iyz="5.41105193e-07" izz="1.41819717e-04"/>
-            </inertial>
-        </link>
-        <joint name="robotiq_camera_joint" type="fixed">
-            <origin xyz="0 0 0" rpy="0 0 0" />
-            <parent link="${parent}"/>
-            <child link="robotiq_camera"/>
-        </joint>
-        <gazebo reference="robotiq_camera">
-            <mu1>0.9</mu1>
-            <mu2>0.9</mu2>
-            <material>Gazebo/Black</material>
-        </gazebo>
         <!-- Robotiq base_link -->
         <link name="${prefix}robotiq_85_base_link">
@@ -60,10 +31,20 @@
             </inertial>
         </link>
-        <joint name="${prefix}robotiq_85_base_joint" type="fixed">
-            <parent link="${prefix}robotiq_camera" />
-            <!-- <parent link="${parent}" /> -->
-            <child link="${prefix}robotiq_85_base_link" />
-            <origin xyz="0 0 13.5e-03" rpy="0 0 0"/>
-        </joint>
+        <xacro:if value="${parent == 'robotiq_camera'}">
+            <joint name="${prefix}robotiq_85_base_joint" type="fixed">
+                <parent link="${parent}" />
+                <!-- <parent link="${parent}" /> -->
+                <child link="${prefix}robotiq_85_base_link" />
+                <origin xyz="0 0 13.5e-03" rpy="0 0 0"/>
+            </joint>
+        </xacro:if>
+        <xacro:unless value="${parent == 'robotiq_camera'}">
+            <joint name="${prefix}robotiq_85_base_joint" type="fixed">
+                <parent link="${parent}" />
+                <!-- <parent link="${parent}" /> -->
+                <child link="${prefix}robotiq_85_base_link" />
+                <origin xyz="0 0 0.0e-03" rpy="0 0 0"/>
+            </joint>
+        </xacro:unless>
         <!-- Robotiq left_knuckle -->
         <link name="${prefix}robotiq_85_left_knuckle_link">
@@ -84,12 +65,22 @@
             </inertial>
         </link>
-        <joint name="${prefix}robotiq_85_left_knuckle_joint" type="revolute">
-            <parent link="${prefix}robotiq_85_base_link" />
-            <child link="${prefix}robotiq_85_left_knuckle_link" />
-            <axis xyz="0 -1 0" />
-            <origin xyz="0.03060114 0.0 0.05490452" rpy="0 0 0" />
-            <limit lower="0.0" upper="0.8" velocity="0.5" effort="50" />
-            <dynamics damping="1.0" friction="1.0"/>
-        </joint>
+        <xacro:if value="${fixed}">
+            <joint name="${prefix}robotiq_85_left_knuckle_joint" type="fixed">
+                <parent link="${prefix}robotiq_85_base_link"/>
+                <child link="${prefix}robotiq_85_left_knuckle_link"/>
+                <origin xyz="0.03060114 0.0 0.05490452" rpy="0 0 0" />
+                <dynamics damping="1.0" friction="1.0"/>
+            </joint>
+        </xacro:if>
+        <xacro:unless value="${fixed}">
+            <joint name="${prefix}robotiq_85_left_knuckle_joint" type="revolute">
+                <parent link="${prefix}robotiq_85_base_link" />
+                <child link="${prefix}robotiq_85_left_knuckle_link" />
+                <axis xyz="0 -1 0" />
+                <origin xyz="0.03060114 0.0 0.05490452" rpy="0 0 0" />
+                <limit lower="0.0" upper="0.8" velocity="0.5" effort="50" />
+                <dynamics damping="1.0" friction="1.0"/>
+            </joint>
+        </xacro:unless>
         <!-- Robotiq right_knuckle -->
         <link name="${prefix}robotiq_85_right_knuckle_link">
@@ -110,13 +101,23 @@
             </inertial>
         </link>
-        <joint name="${prefix}robotiq_85_right_knuckle_joint" type="revolute">
-            <parent link="${prefix}robotiq_85_base_link" />
-            <child link="${prefix}robotiq_85_right_knuckle_link" />
-            <axis xyz="0 -1 0" />
-            <origin xyz="-0.03060114 0.0 0.05490452" rpy="0 0 0" />
-            <limit lower="-0.8" upper="0.0" velocity="0.5" effort="50" />
-            <mimic joint="${prefix}robotiq_85_left_knuckle_joint" multiplier="-1" />
-            <dynamics damping="1.0" friction="1.0"/>
-        </joint>
+        <xacro:if value="${fixed}">
+            <joint name="${prefix}robotiq_85_right_knuckle_joint" type="fixed">
+                <parent link="${prefix}robotiq_85_base_link" />
+                <child link="${prefix}robotiq_85_right_knuckle_link" />
+                <origin xyz="-0.03060114 0.0 0.05490452" rpy="0 0 0" />
+                <dynamics damping="1.0" friction="1.0"/>
+            </joint>
+        </xacro:if>
+        <xacro:unless value="${fixed}">
+            <joint name="${prefix}robotiq_85_right_knuckle_joint" type="revolute">
+                <parent link="${prefix}robotiq_85_base_link" />
+                <child link="${prefix}robotiq_85_right_knuckle_link" />
+                <axis xyz="0 -1 0" />
+                <origin xyz="-0.03060114 0.0 0.05490452" rpy="0 0 0" />
+                <limit lower="-0.8" upper="0.0" velocity="0.5" effort="50" />
+                <mimic joint="${prefix}robotiq_85_left_knuckle_joint" multiplier="-1" />
+                <dynamics damping="1.0" friction="1.0"/>
+            </joint>
+        </xacro:unless>
         <!-- Robotiq left_finger -->
         <link name="${prefix}robotiq_85_left_finger_link">
