Commit message: Finally understood how to move the gripper in gazebo

File: custom_robotiq_description/urdf/robotiq_2f85_ros2_control.xacro (robot description, xacro)
@@ -1,6 +1,6 @@
 <?xml version="1.0"?>
 <robot xmlns:xacro="http://www.ros.org/wiki/xacro">
-    <xacro:macro name="EEF_ros2_control" params="prefix">
-        <joint name="${prefix}robotiq_85_left_knuckle_joint">
+    <xacro:macro name="EEF_ros2_control" params="">
+        <joint name="robotiq_85_left_knuckle_joint">
             <command_interface name="position">
                 <param name="min">-0.05</param>
@@ -17,5 +17,5 @@
             <state_interface name="effort"/>
         </joint>
-        <joint name="${prefix}robotiq_85_right_knuckle_joint">
+        <joint name="robotiq_85_right_knuckle_joint">
             <command_interface name="position">
                 <param name="min">-0.05</param>
@@ -32,5 +32,5 @@
             <state_interface name="effort"/>
         </joint>
-        <joint name="${prefix}robotiq_85_left_inner_knuckle_joint">
+        <joint name="robotiq_85_left_inner_knuckle_joint">
             <command_interface name="position">
                 <param name="min">-0.05</param>
@@ -47,5 +47,5 @@
             <state_interface name="effort"/>
         </joint>
-        <joint name="${prefix}robotiq_85_right_inner_knuckle_joint">
+        <joint name="robotiq_85_right_inner_knuckle_joint">
             <command_interface name="position">
                 <param name="min">-0.05</param>
@@ -62,5 +62,5 @@
             <state_interface name="effort"/>
         </joint>
-        <joint name="${prefix}robotiq_85_left_finger_tip_joint">
+        <joint name="robotiq_85_left_finger_tip_joint">
             <command_interface name="position">
                 <param name="min">-0.80285</param>
@@ -77,5 +77,5 @@
             <state_interface name="effort"/>
         </joint>
-        <joint name="${prefix}robotiq_85_right_finger_tip_joint">
+        <joint name="robotiq_85_right_finger_tip_joint">
             <command_interface name="position">
                 <param name="min">-0.80285</param>

File: custom_ur_description/urdf/custom_ur.urdf.xacro (robot description, xacro)
@@ -50,4 +50,5 @@
    <xacro:arg name="sim_ignition" default="false" />
    <xacro:arg name="simulation_controllers" default="" />
+   <xacro:arg name="use_fixed_gripper" default="false" />
    <!-- initial position for simulations (Fake Hardware, Gazebo, Ignition) -->
    <xacro:arg name="initial_positions_file" default="$(find custom_ur_description)/config/initial_positions.yaml"/>
@@ -98,4 +99,20 @@
      <origin xyz="0 0 0.845" rpy="0 0 0" />          <!-- position robot in the world -->
    </xacro:ur_robot>
+   <!-- <xacro:robotiq_gripper name="RobotiqGripperHardwareInterface" prefix="" parent="$(arg tf_prefix)tool0" use_fake_hardware="$(arg use_fake_hardware)">
+        <origin xyz="0 0 0" rpy="0 0 0" />
+    </xacro:robotiq_gripper> -->
+    <xacro:robotiq_camera prefix="$(arg tf_prefix)" parent="$(arg tf_prefix)tool0"/>
+    <xacro:robotiq_gripper name="RobotiqGripperHardwareInterface" prefix="" parent="robotiq_camera" bringup="false" fixed="$(arg use_fixed_gripper)"/>
+    <!-- END EFFECTOR -->
+    <xacro:unless value="$(arg use_fixed_gripper)">
+      <xacro:include filename="$(find custom_robotiq_description)/urdf/robotiq_2f85_ros2_control.xacro" />
+      <!-- Load ROS2_CONTROL -->
+      <ros2_control name="gripper" type="system">
+        <hardware>
+          <plugin>gazebo_ros2_control/GazeboSystem</plugin>
+        </hardware>
+        <xacro:EEF_ros2_control/>
+      </ros2_control>
+    </xacro:unless>
    <xacro:if value="$(arg sim_gazebo)">
     <!-- Gazebo plugins -->
@@ -107,7 +124,8 @@
         <!-- UR10e Controller -->
         <!-- <parameters>$(arg simulation_controllers)</parameters> -->
-        <parameters>$(find custom_ur_description)/config/ur10e/controller.yaml</parameters>
+        <!-- <parameters>$(find custom_ur_description)/config/ur10e/controller.yaml</parameters> -->
+        <parameters>$(find custom_ur_description)/config/custom_ur_controllers.yaml</parameters>
         <!-- End-Effector Controller (if needed) -->
-        <parameters>$(find custom_robotiq_description)/config/controller.yaml</parameters>
+        <!-- <parameters>$(find custom_robotiq_description)/config/controller.yaml</parameters> -->
       </plugin>
     </gazebo>
@@ -124,8 +142,3 @@
     </gazebo>
   </xacro:if>
-  <!-- <xacro:robotiq_gripper name="RobotiqGripperHardwareInterface" prefix="" parent="$(arg tf_prefix)tool0" use_fake_hardware="$(arg use_fake_hardware)">
-        <origin xyz="0 0 0" rpy="0 0 0" />
-  </xacro:robotiq_gripper> -->
-  <xacro:robotiq_camera prefix="$(arg tf_prefix)" parent="$(arg tf_prefix)tool0"/>
-  <xacro:robotiq_gripper name="RobotiqGripperHardwareInterface" prefix="" parent="robotiq_camera" bringup="$(arg sim_gazebo)" fixed="false"/>
 </robot>
