Commit message: Modified big_bazu and added some urdfs for testing

File: big_bazu/urdf/big_bazu.urdf (robot description, URDF)
Before this commit: robot big_bazu, 2 links, 1 joints
Links:
- added link link_1, mass 5.0; collision cylinder length=0.5 radius=0.08; visual cylinder length=0.5 radius=0.08
- added link link_2, mass 2.0; collision cylinder length=0.1 radius=0.08; visual cylinder length=0.1 radius=0.08
- added link link_3, mass 1.0; collision cylinder length=0.4 radius=0.05; visual cylinder length=0.4 radius=0.05
- link base_link: mass None -> 5.0; geometry collision cylinder length=0.05 radius=0.2; visual cylinder length=0.05 radius=0.2
Joints:
- removed joint base_joint
- added joint fixed: type fixed, parent world, child base_link
- added joint joint_1: type continuous, parent base_link, child link_1, origin xyz=0.0 0.0 0.05 rpy=0 0 0, axis 0 0 1
- added joint joint_2: type revolute, parent link_1, child link_2, origin xyz=0.0 -0.005 0.58 rpy=0 1.5708 0, axis 0 0 1, limit lower=-0.25 upper=3.34 effort=10 velocity=0.5
- added joint joint_3: type fixed, parent link_2, child link_3, origin xyz=0.0 0.2 0  rpy=1.57 0 0
