Commit message: Modified the joint limits of Mark 1

File: mark_one_arm_description/urdf/mark_one_arm.urdf.xacro (robot description, xacro)
@@ -3,5 +3,5 @@
      Commit Version: 1.6.0-4-g7f85cfe  Build Version: 1.6.7995.38578
      For more information, please see http://wiki.ros.org/sw_urdf_exporter -->
-<robot name="mark_one_arm">
+<robot name="mark_one_arm" xmlns:xacro="http://www.ros.org/wiki/xacro">
   <!-- create link fixed to the "world" -->
   <link name="world" />
@@ -73,5 +73,5 @@
     <child link="Link_1" />
     <axis xyz="0 0 -1" />
-    <limit lower="0" upper="4.18" effort="1" velocity="3" />
+    <limit lower="-${pi}" upper="${pi}" effort="1" velocity="3" />
   </joint>
   <link name="Link_2">
@@ -108,5 +108,5 @@
     <child link="Link_2" />
     <axis xyz="0 1 0" />
-    <limit lower="0" upper="4.18" effort="1" velocity="3" />
+    <limit lower="-${pi/2}" upper="${pi/2}" effort="1" velocity="3" />
   </joint>
   <link name="Link_3">
@@ -143,5 +143,5 @@
     <child link="Link_3" />
     <axis xyz="0 1 0" />
-    <limit lower="0" upper="4.18" effort="1" velocity="3" />
+    <limit lower="-${pi/2}" upper="${pi/2}" effort="1" velocity="3" />
   </joint>
   <link name="Link_4">
@@ -178,5 +178,5 @@
     <child link="Link_4" />
     <axis xyz="1 0 0" />
-    <limit lower="-0.52" upper="2.62" effort="0.118" velocity="4.2" />
+    <limit lower="-${pi}" upper="${pi}" effort="0.118" velocity="4.2" />
   </joint>
   <link name="Link_5">
@@ -213,5 +213,5 @@
     <child link="Link_5" />
     <axis xyz="0 -1 0" />
-    <limit lower="-0.52" upper="2.62" effort="0.118" velocity="4.2" />
+    <limit lower="-${pi}" upper="${pi}" effort="0.118" velocity="4.2" />
   </joint>
 </robot>

Commit message: Creating the integration with gazebo

File: mark_one_arm_description/urdf/mark_one_arm.urdf.xacro (robot description, xacro)
@@ -4,4 +4,14 @@
      For more information, please see http://wiki.ros.org/sw_urdf_exporter -->
 <robot name="mark_one_arm" xmlns:xacro="http://www.ros.org/wiki/xacro">
+  <xacro:arg name="sim_gazebo" default="false" />
+  <xacro:arg name="sim_ignition" default="false" />
+  <!-- initial position for simulations (Fake Hardware, Gazebo, Ignition) -->
+  <xacro:arg name="initial_positions_file" default="$(find mark_one_arm_description)/config/initial_positions.yaml"/>
+  <xacro:include filename="$(find mark_one_arm_description)/urdf/mark_one_gazebo.xacro"/>
+  <xacro:include filename="$(find mark_one_arm_description)/urdf/mark_one_ros2_control.xacro"/>
+   <!-- convert to property to use substitution in function -->
+  <xacro:property name="initial_positions_file" default="$(arg initial_positions_file)"/>
+  <xacro:property name="effort" value="1.5"/>
+  <xacro:property name="velocity" value="${2*pi}"/>
   <!-- create link fixed to the "world" -->
   <link name="world" />
@@ -68,10 +78,10 @@
     </collision>
   </link>
-  <joint name="Joint_1" type="revolute">
+  <joint name="joint_1" type="revolute">
     <origin xyz="0.0005 0 0.0675" rpy="0 0 3.1416" />
     <parent link="base_link" />
     <child link="Link_1" />
     <axis xyz="0 0 -1" />
-    <limit lower="-${pi}" upper="${pi}" effort="1" velocity="3" />
+    <limit lower="-${pi}" upper="${pi}" effort="${effort}" velocity="${velocity}" />
   </joint>
   <link name="Link_2">
@@ -103,10 +113,10 @@
     </collision>
   </link>
-  <joint name="Joint_2" type="revolute">
+  <joint name="joint_2" type="revolute">
     <origin xyz="0.0005 -0.00615 0.0875" rpy="0 0 0" />
     <parent link="Link_1" />
     <child link="Link_2" />
     <axis xyz="0 1 0" />
-    <limit lower="-${pi/2}" upper="${pi/2}" effort="1" velocity="3" />
+    <limit lower="-${pi/2}" upper="${pi/2}" effort="${effort}" velocity="${velocity}" />
   </joint>
   <link name="Link_3">
@@ -138,10 +148,10 @@
     </collision>
   </link>
-  <joint name="Joint_3" type="revolute">
+  <joint name="joint_3" type="revolute">
     <origin xyz="0 0 0.20005" rpy="0 0 0" />
     <parent link="Link_2" />
     <child link="Link_3" />
     <axis xyz="0 1 0" />
-    <limit lower="-${pi/2}" upper="${pi/2}" effort="1" velocity="3" />
+    <limit lower="-${pi/2}" upper="${pi/2}" effort="${effort}" velocity="${velocity}" />
   </joint>
   <link name="Link_4">
@@ -173,10 +183,10 @@
     </collision>
   </link>
-  <joint name="Joint_4" type="revolute">
+  <joint name="joint_4" type="revolute">
     <origin xyz="-0.15685 -0.0252 0.0054" rpy="0 0 0" />
     <parent link="Link_3" />
     <child link="Link_4" />
     <axis xyz="1 0 0" />
-    <limit lower="-${pi}" upper="${pi}" effort="0.118" velocity="4.2" />
+    <limit lower="-${pi}" upper="${pi}" effort="${effort}" velocity="${velocity}" />
   </joint>
   <link name="Link_5">
@@ -208,10 +218,10 @@
     </collision>
   </link>
-  <joint name="Joint_5" type="revolute">
+  <joint name="joint_5" type="revolute">
     <origin xyz="-0.03875 0.02745 -0.00545" rpy="0 0 0" />
     <parent link="Link_4" />
     <child link="Link_5" />
     <axis xyz="0 -1 0" />
-    <limit lower="-${pi}" upper="${pi}" effort="0.118" velocity="4.2" />
+    <limit lower="-${pi}" upper="${pi}" effort="${effort}" velocity="${velocity}" />
   </joint>
 </robot>

Commit message: Integration with classic gazebo complete, working on adjusting the inertial of the base

File: mark_one_arm_description/urdf/mark_one_arm.urdf.xacro (robot description, xacro)
@@ -8,10 +8,11 @@
   <!-- initial position for simulations (Fake Hardware, Gazebo, Ignition) -->
   <xacro:arg name="initial_positions_file" default="$(find mark_one_arm_description)/config/initial_positions.yaml"/>
+  <!-- convert to property to use substitution in function -->
+  <xacro:property name="initial_positions_file" default="$(arg initial_positions_file)"/>
+  <xacro:property name="initial_positions" value="${xacro.load_yaml(initial_positions_file)}"/>
+  <xacro:property name="effort" value="1.5"/>
+  <xacro:property name="velocity" value="${2*pi}"/>
   <xacro:include filename="$(find mark_one_arm_description)/urdf/mark_one_gazebo.xacro"/>
   <xacro:include filename="$(find mark_one_arm_description)/urdf/mark_one_ros2_control.xacro"/>
-   <!-- convert to property to use substitution in function -->
-  <xacro:property name="initial_positions_file" default="$(arg initial_positions_file)"/>
-  <xacro:property name="effort" value="1.5"/>
-  <xacro:property name="velocity" value="${2*pi}"/>
   <!-- create link fixed to the "world" -->
   <link name="world" />
@@ -31,5 +32,5 @@
       <origin xyz="0 0 0" rpy="0 0 0" />
       <geometry>
-        <mesh filename="package://mark_one_arm_description/meshes/base_link.STL" />
+        <mesh filename="file://$(find mark_one_arm_description)/meshes/base_link.STL" />
           <!-- filename="package://AMH19_Mark1_Complete_URDF/meshes/base_link.STL" />  -->
       </geometry>
@@ -39,7 +40,8 @@
     </visual>
     <collision>
-      <origin xyz="0 0 0" rpy="0 0 0" />
-      <geometry>
-        <mesh filename="package://mark_one_arm_description/meshes/base_link.STL" />
+      <origin xyz="0 0 0.03" rpy="0 0 0" />
+      <geometry>
+        <!-- <mesh filename="package://mark_one_arm_description/meshes/base_link.STL" /> -->
+        <box size="0.2074 0.2074 0.07"/>
       </geometry>
     </collision>
@@ -48,5 +50,5 @@
     <parent link="world"/>
     <child link="base_link"/>
-    <origin rpy="0.0 0.0 0.0" xyz="0.0 0.0 0.0"/>
+    <origin rpy="0.0 0.0 0.0" xyz="0.0 0.0 0.005"/>
   </joint>
   <link name="Link_1">
@@ -65,14 +67,14 @@
       <origin xyz="0 0 0" rpy="0 0 0" />
       <geometry>
-        <mesh filename="package://mark_one_arm_description/meshes/Link_1.STL" />
-      </geometry>
-      <material name="">
-        <color rgba="0.19608 0.58824 1 1" />
-      </material>
-    </visual>
-    <collision>
-      <origin xyz="0 0 0" rpy="0 0 0" />
-      <geometry>
-        <mesh filename="package://mark_one_arm_description/meshes/Link_1.STL" />
+        <mesh filename="file://$(find mark_one_arm_description)/meshes/Link_1.STL" />
+      </geometry>
+      <material name="">
+        <color rgba="0.19608 0.58824 1 1" />
+      </material>
+    </visual>
+    <collision>
+      <origin xyz="0 0 0" rpy="0 0 0" />
+      <geometry>
+        <mesh filename="file://$(find mark_one_arm_description)/meshes/Link_1.STL" />
       </geometry>
     </collision>
@@ -100,14 +102,14 @@
       <origin xyz="0 0 0" rpy="0 0 0" />
       <geometry>
-        <mesh filename="package://mark_one_arm_description/meshes/Link_2.STL" />
-      </geometry>
-      <material name="">
-        <color rgba="0.19608 0.58824 1 1" />
-      </material>
-    </visual>
-    <collision>
-      <origin xyz="0 0 0" rpy="0 0 0" />
-      <geometry>
-        <mesh filename="package://mark_one_arm_description/meshes/Link_2.STL" />
+        <mesh filename="file://$(find mark_one_arm_description)/meshes/Link_2.STL" />
+      </geometry>
+      <material name="">
+        <color rgba="0.19608 0.58824 1 1" />
+      </material>
+    </visual>
+    <collision>
+      <origin xyz="0 0 0" rpy="0 0 0" />
+      <geometry>
+        <mesh filename="file://$(find mark_one_arm_description)/meshes/Link_2.STL" />
       </geometry>
     </collision>
@@ -135,14 +137,14 @@
       <origin xyz="0 0 0" rpy="0 0 0" />
       <geometry>
-        <mesh filename="package://mark_one_arm_description/meshes/Link_3.STL" />
-      </geometry>
-      <material name="">
-        <color rgba="0.19608 0.58824 1 1" />
-      </material>
-    </visual>
-    <collision>
-      <origin xyz="0 0 0" rpy="0 0 0" />
-      <geometry>
-        <mesh filename="package://mark_one_arm_description/meshes/Link_3.STL" />
+        <mesh filename="file://$(find mark_one_arm_description)/meshes/Link_3.STL" />
+      </geometry>
+      <material name="">
+        <color rgba="0.19608 0.58824 1 1" />
+      </material>
+    </visual>
+    <collision>
+      <origin xyz="0 0 0" rpy="0 0 0" />
+      <geometry>
+        <mesh filename="file://$(find mark_one_arm_description)/meshes/Link_3.STL" />
       </geometry>
     </collision>
@@ -170,14 +172,14 @@
       <origin xyz="0 0 0" rpy="0 0 0" />
       <geometry>
-        <mesh filename="package://mark_one_arm_description/meshes/Link_4.STL" />
-      </geometry>
-      <material name="">
-        <color rgba="0.19608 0.58824 1 1" />
-      </material>
-    </visual>
-    <collision>
-      <origin xyz="0 0 0" rpy="0 0 0" />
-      <geometry>
-        <mesh filename="package://mark_one_arm_description/meshes/Link_4.STL" />
+        <mesh filename="file://$(find mark_one_arm_description)/meshes/Link_4.STL" />
+      </geometry>
+      <material name="">
+        <color rgba="0.19608 0.58824 1 1" />
+      </material>
+    </visual>
+    <collision>
+      <origin xyz="0 0 0" rpy="0 0 0" />
+      <geometry>
+        <mesh filename="file://$(find mark_one_arm_description)/meshes/Link_4.STL" />
       </geometry>
     </collision>
@@ -205,14 +207,14 @@
       <origin xyz="0 0 0" rpy="0 0 0" />
       <geometry>
-        <mesh filename="package://mark_one_arm_description/meshes/Link_5.STL" />
-      </geometry>
-      <material name="">
-        <color rgba="0.19608 0.58824 1 1" />
-      </material>
-    </visual>
-    <collision>
-      <origin xyz="0 0 0" rpy="0 0 0" />
-      <geometry>
-        <mesh filename="package://mark_one_arm_description/meshes/Link_5.STL" />
+        <mesh filename="file://$(find mark_one_arm_description)/meshes/Link_5.STL" />
+      </geometry>
+      <material name="">
+        <color rgba="0.19608 0.58824 1 1" />
+      </material>
+    </visual>
+    <collision>
+      <origin xyz="0 0 0" rpy="0 0 0" />
+      <geometry>
+        <mesh filename="file://$(find mark_one_arm_description)/meshes/Link_5.STL" />
       </geometry>
     </collision>

File: mark_one_arm_description/urdf/mark_one_gazebo.xacro (robot description, xacro)
@@ -1,10 +1,13 @@
 <?xml version="1.0"?>
-<robot xmlns:xacro="http://www.ros.org/wiki/xacro">
-   <xacro:if value="$(arg sim_gazebo)">
+<robot xmlns:xacro="http://www.ros.org/wiki/xacro" name="mark_one_arm">
+  <gazebo reference="Link_1">
+        <material>Gazebo/Green</material>
+  </gazebo>
+  <xacro:if value="$(arg sim_gazebo)">
     <!-- Gazebo plugins -->
     <gazebo reference="world"/>
     <gazebo>
       <plugin filename="libgazebo_ros2_control.so" name="gazebo_ros2_control">
-        <parameters>$(arg simulation_controllers)</parameters>
+        <parameters>$(find mark_one_arm_description)/config/mark_one_controllers.yaml</parameters>
       </plugin>
     </gazebo>
@@ -15,6 +18,6 @@
     <gazebo>
       <plugin filename="libign_ros2_control-system.so" name="ign_ros2_control::IgnitionROS2ControlPlugin">
-        <parameters>$(arg simulation_controllers)</parameters>
-        <controller_manager_node_name>$(arg tf_prefix)controller_manager</controller_manager_node_name>
+        <parameters>$(find mark_one_arm_description)/config/mark_one_controllers.yaml</parameters>
+        <!-- <controller_manager_node_name>$(arg tf_prefix)controller_manager</controller_manager_node_name> -->
       </plugin>
     </gazebo>

File: mark_one_arm_description/urdf/mark_one_ros2_control.xacro (robot description, xacro)
@@ -1,73 +1,73 @@
 <?xml version="1.0"?>
-<robot xmlns:xacro="http://www.ros.org/wiki/xacro">
+<robot xmlns:xacro="http://www.ros.org/wiki/xacro" name="mark_one_arm">
     <ros2_control type="system" name="RobotSystem">
         <hardware>
-            <xacro:if value="${sim_gazebo}">
+            <xacro:if value="$(arg sim_gazebo)">
                 <plugin>gazebo_ros2_control/GazeboSystem</plugin>
             </xacro:if>
-            <xacro:if value="${sim_ignition}">
+            <xacro:if value="$(arg sim_ignition)">
                 <plugin>ign_ros2_control/IgnitionSystem</plugin>
             </xacro:if>
         </hardware>
+        <joint name="joint_1">
+            <command_interface name="position"/>
+                <param name="min"> -${pi} </param>
+                <param name="min"> ${pi} </param>
+            <command_interface name="velocity"/>
+            <state_interface name="position">
+                <!-- initial position for the FakeSystem and simulation -->
+                <param name="initial_value">${initial_positions['joint_1']}</param>
+            </state_interface>
+            <state_interface name="velocity"/>
+            <state_interface name="effort"/>
+        </joint>
+        <joint name="joint_2">
+            <command_interface name="position"/>
+                <param name="min"> -${pi/2} </param>
+                <param name="min"> ${pi/2} </param>
+            <command_interface name="velocity"/>
+            <state_interface name="position">
+                <!-- initial position for the FakeSystem and simulation -->
+                <param name="initial_value">${initial_positions['joint_2']}</param>
+            </state_interface>
+            <state_interface name="velocity"/>
+            <state_interface name="effort"/>
+        </joint>
+        <joint name="joint_3">
+            <command_interface name="position"/>
+                <param name="min"> -${pi/2} </param>
+                <param name="min"> ${pi/2} </param>
+            <command_interface name="velocity"/>
+            <state_interface name="position">
+                <!-- initial position for the FakeSystem and simulation -->
+                <param name="initial_value">${initial_positions['joint_3']}</param>
+            </state_interface>
+            <state_interface name="velocity"/>
+            <state_interface name="effort"/>
+        </joint>
+        <joint name="joint_4">
+            <command_interface name="position"/>
+                <param name="min"> -${pi} </param>
+                <param name="min"> ${pi} </param>
+            <command_interface name="velocity"/>
+            <state_interface name="position">
+                <!-- initial position for the FakeSystem and simulation -->
+                <param name="initial_value">${initial_positions['joint_4']}</param>
+            </state_interface>
+            <state_interface name="velocity"/>
+            <state_interface name="effort"/>
+        </joint>
+        <joint name="joint_5">
+            <command_interface name="position"/>
+                <param name="min"> -${pi} </param>
+                <param name="min"> ${pi} </param>
+            <command_interface name="velocity"/>
+            <state_interface name="position">
+                <!-- initial position for the FakeSystem and simulation -->
+                <param name="initial_value">${initial_positions['joint_5']}</param>
+            </state_interface>
+            <state_interface name="velocity"/>
+            <state_interface name="effort"/>
+        </joint>
     </ros2_control>
-    <joint name="joint_1">
-        <command_interface name="position"/>
-            <param name="min"> -${pi} </param>
-            <param name="min"> ${pi} </param>
-        <command_interface name="velocity"/>
-        <state_interface name="position">
-          <!-- initial position for the FakeSystem and simulation -->
-          <param name="initial_value">${initial_positions['joint_1']}</param>
-        </state_interface>
-        <state_interface name="velocity"/>
-        <state_interface name="effort"/>
-    </joint>
-    <joint name="joint_2">
-        <command_interface name="position"/>
-            <param name="min"> -${pi/2} </param>
-            <param name="min"> ${pi/2} </param>
-        <command_interface name="velocity"/>
-        <state_interface name="position">
-          <!-- initial position for the FakeSystem and simulation -->
-          <param name="initial_value">${initial_positions['joint_2']}</param>
-        </state_interface>
-        <state_interface name="velocity"/>
-        <state_interface name="effort"/>
-    </joint>
-    <joint name="joint_3">
-        <command_interface name="position"/>
-            <param name="min"> -${pi/2} </param>
-            <param name="min"> ${pi/2} </param>
-        <command_interface name="velocity"/>
-        <state_interface name="position">
-          <!-- initial position for the FakeSystem and simulation -->
-          <param name="initial_value">${initial_positions['joint_3']}</param>
-        </state_interface>
-        <state_interface name="velocity"/>
-        <state_interface name="effort"/>
-    </joint>
-    <joint name="joint_4">
-        <command_interface name="position"/>
-            <param name="min"> -${pi} </param>
-            <param name="min"> ${pi} </param>
-        <command_interface name="velocity"/>
-        <state_interface name="position">
-          <!-- initial position for the FakeSystem and simulation -->
-          <param name="initial_value">${initial_positions['joint_4']}</param>
-        </state_interface>
-        <state_interface name="velocity"/>
-        <state_interface name="effort"/>
-    </joint>
-    <joint name="joint_5">
-        <command_interface name="position"/>
-            <param name="min"> -${pi} </param>
-            <param name="min"> ${pi} </param>
-        <command_interface name="velocity"/>
-        <state_interface name="position">
-          <!-- initial position for the FakeSystem and simulation -->
-          <param name="initial_value">${initial_positions['joint_5']}</param>
-        </state_interface>
-        <state_interface name="velocity"/>
-        <state_interface name="effort"/>
-    </joint>
 </robot>

Commit message: Fixed base inertia

File: mark_one_arm_description/urdf/mark_one_arm.urdf.xacro (robot description, xacro)
@@ -13,4 +13,5 @@
   <xacro:property name="effort" value="1.5"/>
   <xacro:property name="velocity" value="${2*pi}"/>
+  <xacro:include filename="$(find mark_one_arm_description)/urdf/common_properties.xacro"/>
   <xacro:include filename="$(find mark_one_arm_description)/urdf/mark_one_gazebo.xacro"/>
   <xacro:include filename="$(find mark_one_arm_description)/urdf/mark_one_ros2_control.xacro"/>
@@ -18,5 +19,6 @@
   <link name="world" />
   <link name="base_link">
-    <inertial>
+    <xacro:box_inertia m="1.7609" l="0.2074" w="0.2074" h="0.07" xyz="0 0 0.03" rpy="${pi/2} 0 0"/>
+    <!-- <inertial>
       <origin xyz="-0.038112 1.1649E-05 -0.051288" rpy="0 0 0" />
       <mass value="1.7609" />
@@ -28,5 +30,5 @@
         iyz="-1.5817E-06"
         izz="0.0096448" />
-    </inertial>
+    </inertial> -->
     <visual>
       <origin xyz="0 0 0" rpy="0 0 0" />
