Commit message: editing big_bazu to make it more functional

File: big_bazu_description/urdf/big_bazu.urdf (robot description, URDF)
Before this commit: robot big_bazu, 5 links, 4 joints
Links:
- added link link_2_body, mass 1.0; collision cylinder length=0.4 radius=0.05; visual cylinder length=0.4 radius=0.05
- added link link_3_body, mass 1.0; collision cylinder length=0.3 radius=0.04; visual cylinder length=0.3 radius=0.04
- link link_2: geometry collision cylinder length=0.3 radius=0.08; visual cylinder length=0.3 radius=0.08
- link link_3: mass 1.0 -> 2.0; geometry collision cylinder length=0.2 radius=0.05; visual cylinder length=0.2 radius=0.05
Joints:
- added joint fixed_joint_1: type fixed, parent link_2, child link_2_body, origin xyz=0.2 0.0 0  rpy=0 1.5708 0
- added joint fixed_joint_2: type fixed, parent link_3, child link_3_body, origin xyz=0.15 0.0 0.095  rpy=0 1.5708 0
- joint joint_1: limit (none) -> lower=-6.2832 upper=6.2832 effort=0.0 velocity=0.0; type continuous -> revolute
- joint joint_2: limit lower=-0.25 upper=3.34 effort=10 velocity=0.5 -> lower=-3.1416 upper=3.1416 effort=10 velocity=0.5; origin xyz=0.0 -0.005 0.58 rpy=0 1.5708 0 -> xyz=0.0 0.15 0.58 rpy=1.5708 0.0 0.0
- joint joint_3: axis (none) -> 0 0 1; limit (none) -> lower=-0.25 upper=3.34 effort=10 velocity=0.5; origin xyz=0.0 0.2 0  rpy=1.57 0 0 -> xyz=0.425 0.0 0.0 rpy=0 0 0; type fixed -> revolute
