Commit message: working on the differential robot for the summer course

File: diff_summer_robot_description/urdf/diff_summer_robot.urdf (robot description, URDF)
Before this commit: robot diff_summer_robot, 1 links, 0 joints
Links:
- added link right_wheel_link; visual cylinder length=0.05 radius=0.1
- link base_link: geometry visual box size=0.6 0.4 0.2
Joints:
- added joint base_right_wheel_joint: type continuous, parent base_link, child right_wheel_link, origin xyz=-0.15 -0.225 0.0 rpy=0.0 0.0 0.0, axis 0 1 0
