Commit message: Improved summer robot description with xacro

File: diff_summer_robot_description/urdf/diff_summer_robot_tutor.urdf.xacro (robot description, xacro)
@@ -1,4 +1,9 @@
 <?xml version="1.0" encoding="UTF-8"?>
-<robot name="my_tutor_robot">
+<robot name="my_tutor_robot" xmlns:xacro="http://www.ros.org/wiki/xacro">
+    <xacro:property name="base_length" value="0.6"/>
+    <xacro:property name="base_width" value="0.4"/>
+    <xacro:property name="base_height" value="0.2"/>
+    <xacro:property name="wheel_radius" value="0.1"/>
+    <xacro:property name="wheel_length" value="0.05"/>
     <material name="green">
         <color rgba="0.0 0.5 0.0 1.0"/>
@@ -11,5 +16,5 @@
         <visual>
             <geometry>
-                <box size="0.6 0.4 0.2"/>
+                <box size="${base_length} ${base_width} ${base_height}"/>
             </geometry>
             <origin xyz="0.0 0.0 0.1" rpy="0.0 0.0 0.0"/>
@@ -37,7 +42,7 @@
     <link name="right_wheel_link">
         <visual>
-            <origin xyz="0.0 0.0 0.0" rpy="1.57 0.0 0.0"/>
+            <origin xyz="0.0 0.0 0.0" rpy="${pi / 2} 0.0 0.0"/>
             <geometry>
-                <cylinder radius="0.1" length="0.05"/>
+                <cylinder radius="${wheel_radius}" length="${wheel_length}"/>
             </geometry>
             <material name="grey"/>
@@ -46,7 +51,7 @@
     <link name="left_wheel_link">
         <visual>
-            <origin xyz="0.0 0.0 0.0" rpy="1.57 0.0 0.0"/>
+            <origin xyz="0.0 0.0 0.0" rpy="${pi / 2} 0.0 0.0"/>
             <geometry>
-                <cylinder radius="0.1" length="0.05"/>
+                <cylinder radius="${wheel_radius}" length="${wheel_length}"/>
             </geometry>
             <material name="grey"/>
@@ -57,5 +62,5 @@
             <origin xyz="0.0 0.0 0.0" rpy="0.0 0.0 0.0"/>
             <geometry>
-                <sphere radius="0.05"/>
+                <sphere radius="${wheel_radius/2.0}"/>
             </geometry>
             <material name="grey"/>
@@ -84,5 +89,5 @@
         <parent link="base_link"/>
         <child link="right_wheel_link"/>
-        <origin xyz="-0.15 -0.225 0.0" rpy="0.0 0.0 0.0"/>
+        <origin xyz="${-base_length / 4.0} ${-((base_width/2.0)+(wheel_length/2.0))} 0.0" rpy="0.0 0.0 0.0"/>
         <axis xyz="0 1 0"/>
     </joint>
@@ -91,10 +96,10 @@
         <child link="left_wheel_link"/>
         <axis xyz="0 1 0"/>
-        <origin xyz="-0.15 0.225 0" rpy="0 0 0"/>
+        <origin xyz="${-base_length / 4.0} ${(base_width/2.0)+(wheel_length/2.0)} 0" rpy="0 0 0"/>
     </joint>
     <joint name="base_caster_wheel_joint" type="fixed">
         <parent link="base_link"/>
         <child link="caster_wheel_link"/>
-        <origin xyz="0.2 0.0 -0.05" rpy="0.0 0.0 0.0"/>
+        <origin xyz="${base_length / 3.0} 0.0 ${-wheel_radius/2.0}" rpy="0.0 0.0 0.0"/>
     </joint>
 </robot>

Commit message: tutorial robot improvement

File: diff_summer_robot_description/urdf/diff_summer_robot_tutor.urdf.xacro (robot description, xacro)
@@ -1,105 +1,5 @@
 <?xml version="1.0" encoding="UTF-8"?>
 <robot name="my_tutor_robot" xmlns:xacro="http://www.ros.org/wiki/xacro">
-    <xacro:property name="base_length" value="0.6"/>
-    <xacro:property name="base_width" value="0.4"/>
-    <xacro:property name="base_height" value="0.2"/>
-    <xacro:property name="wheel_radius" value="0.1"/>
-    <xacro:property name="wheel_length" value="0.05"/>
-    <material name="green">
-        <color rgba="0.0 0.5 0.0 1.0"/>
-    </material>
-    <material name="grey">
-        <color rgba="0.5 0.5 0.5 1.0"/>
-    </material>
-    <link name="base_footprint"/>
-    <link name="base_link">
-        <visual>
-            <geometry>
-                <box size="${base_length} ${base_width} ${base_height}"/>
-            </geometry>
-            <origin xyz="0.0 0.0 0.1" rpy="0.0 0.0 0.0"/>
-            <material name="green"/>
-        </visual>
-    </link>
-    <!-- <link name="second_link">
-        <visual>
-            <geometry>
-                <cylinder radius="0.1" length="0.2"/>
-            </geometry>
-            <origin xyz="0.0 0.0 0.1" rpy="0.0 0.0 0.0"/>
-            <material name="grey"/>
-        </visual>
-    </link>
-    <link name="third_link">
-        <visual>
-            <origin xyz="0.0 0.0 0.05" rpy="0.0 0.0 0.0"/>
-            <geometry>
-                <box size="0.1 0.1 0.1"/>
-            </geometry>
-            <material name="green"/>
-        </visual>
-    </link> -->
-    <link name="right_wheel_link">
-        <visual>
-            <origin xyz="0.0 0.0 0.0" rpy="${pi / 2} 0.0 0.0"/>
-            <geometry>
-                <cylinder radius="${wheel_radius}" length="${wheel_length}"/>
-            </geometry>
-            <material name="grey"/>
-        </visual>
-    </link>
-    <link name="left_wheel_link">
-        <visual>
-            <origin xyz="0.0 0.0 0.0" rpy="${pi / 2} 0.0 0.0"/>
-            <geometry>
-                <cylinder radius="${wheel_radius}" length="${wheel_length}"/>
-            </geometry>
-            <material name="grey"/>
-        </visual>
-    </link>
-    <link name="caster_wheel_link">
-        <visual>
-            <origin xyz="0.0 0.0 0.0" rpy="0.0 0.0 0.0"/>
-            <geometry>
-                <sphere radius="${wheel_radius/2.0}"/>
-            </geometry>
-            <material name="grey"/>
-        </visual>
-    </link>
-    <!-- <joint name="base_second_joint" type="revolute">
-        <parent link="base_link"/>
-        <child link="second_link"/>
-        <axis xyz="0 0 1"/>
-        <limit lower="-1.57" upper="1.57" effort="1.0" velocity="3.14"/>
-        <origin xyz="0.0 0.0 0.2" rpy="0.0 0.0 0.0"/>
-    </joint>
-    <joint name="second_third_joint" type="prismatic">
-        <parent link="second_link"/>
-        <child link="third_link"/>
-        <origin xyz="0.0 0.0 0.2" rpy="0.0 0.0 0.0"/>
-        <axis xyz="0 0 1"/>
-        <limit lower="0.0" upper="0.2" effort="1.0" velocity="0.1"/>
-    </joint> -->
-    <joint name="base_joint" type="fixed">
-        <parent link="base_footprint"/>
-        <child link="base_link"/>
-        <origin xyz="0.0 0.0 0.1" rpy="0.0 0.0 0.0"/>
-    </joint>
-    <joint name="base_right_wheel_joint" type="continuous">
-        <parent link="base_link"/>
-        <child link="right_wheel_link"/>
-        <origin xyz="${-base_length / 4.0} ${-((base_width/2.0)+(wheel_length/2.0))} 0.0" rpy="0.0 0.0 0.0"/>
-        <axis xyz="0 1 0"/>
-    </joint>
-    <joint name="base_left_wheel_joint" type="continuous">
-        <parent link="base_link"/>
-        <child link="left_wheel_link"/>
-        <axis xyz="0 1 0"/>
-        <origin xyz="${-base_length / 4.0} ${(base_width/2.0)+(wheel_length/2.0)} 0" rpy="0 0 0"/>
-    </joint>
-    <joint name="base_caster_wheel_joint" type="fixed">
-        <parent link="base_link"/>
-        <child link="caster_wheel_link"/>
-        <origin xyz="${base_length / 3.0} 0.0 ${-wheel_radius/2.0}" rpy="0.0 0.0 0.0"/>
-    </joint>
+    <xacro:include filename="$(find diff_summer_robot_description)/urdf/common_properties_tutor.xacro"/>
+    <xacro:include filename="$(find diff_summer_robot_description)/urdf/mobile_base_tutor.xacro"/>
 </robot>
