Commit message: Not sure why but the gazebo plugins does not seem to work

File: diff_summer_robot_description/urdf/common_properties_tutor.xacro (robot description, xacro)
@@ -14,3 +14,17 @@
         </inertial>
     </xacro:macro>
+    <xacro:macro name="cylinder_inertia" params="m r l o_xyz o_rpy">
+        <inertial>
+            <origin xyz="${o_xyz}" rpy="${o_rpy}"/>
+            <mass value="${m}"/>
+            <inertia ixx="${(m/12.0) * (l*l + 3.0*r*r)}" ixy="0.0" ixz="0.0" iyy="${(m/12.0) * (l*l + 3.0*r*r)}" iyz="0.0" izz="${(m/2.0) * (r*r)}"/>
+        </inertial>
+    </xacro:macro>
+    <xacro:macro name="sphere_inertia" params="m r o_xyz o_rpy">
+        <inertial>
+            <origin xyz="${o_xyz}" rpy="${o_rpy}"/>
+            <mass value="${m}"/>
+            <inertia ixx="${(2.0*m/5.0) * (r*r)}" ixy="0.0" ixz="0.0" iyy="${(2.0*m/5.0) * (r*r)}" iyz="0.0" izz="${(2.0*m/5.0) * (r*r)}"/>
+        </inertial>
+    </xacro:macro>
 </robot>

File: diff_summer_robot_description/urdf/diff_summer_robot_tutor.urdf.xacro (robot description, xacro)
@@ -3,3 +3,4 @@
     <xacro:include filename="$(find diff_summer_robot_description)/urdf/common_properties_tutor.xacro"/>
     <xacro:include filename="$(find diff_summer_robot_description)/urdf/mobile_base_tutor.xacro"/>
+    <xacro:include filename="$(find diff_summer_robot_description)/urdf/mobile_base_gazebo_tutor.xacro"/>
 </robot>

File: diff_summer_robot_description/urdf/mobile_base_tutor.xacro (robot description, xacro)
@@ -8,4 +8,5 @@
     <xacro:macro name="wheel_link" params="prefix">
         <link name="${prefix}_wheel_link">
+            <xacro:cylinder_inertia m="1.0" r="${wheel_radius}" l="${wheel_length}" o_xyz="0.0 0.0 0.0" o_rpy="${pi/2.0} 0.0 0.0"/>
             <visual>
                 <origin xyz="0.0 0.0 0.0" rpy="${pi / 2.0} 0.0 0.0"/>
@@ -15,4 +16,10 @@
                 <material name="grey"/>
             </visual>
+            <collision>
+                <origin xyz="0.0 0.0 0.0" rpy="${pi / 2.0} 0.0 0.0"/>
+                <geometry>
+                    <sphere radius="${wheel_radius}"/>
+                </geometry>
+            </collision>
         </link>
     </xacro:macro>
@@ -29,8 +36,16 @@
             <material name="green"/>
         </visual>
+        <collision>
+            <origin xyz="0.0 0.0 ${base_height/ 2.0}" rpy="0.0 0.0 0.0"/>
+            <geometry>
+                <box size="${base_length} ${base_width} ${base_height}"/>
+            </geometry>
+        </collision>
     </link>
     <xacro:wheel_link prefix="right"/>
     <xacro:wheel_link prefix="left"/>
     <link name="caster_wheel_link">
+        <xacro:sphere_inertia m="0.5" r="${wheel_radius/2.0}"
+                           o_xyz="0.0 0.0 0.0" o_rpy="0.0 0.0 0.0"/>
         <visual>
             <origin xyz="0.0 0.0 0.0" rpy="0.0 0.0 0.0"/>
@@ -40,4 +55,10 @@
             <material name="grey"/>
         </visual>
+        <collision>
+            <origin xyz="0.0 0.0 0.0" rpy="0.0 0.0 0.0"/>
+            <geometry>
+                <sphere radius="${wheel_radius / 2.0}"/>
+            </geometry>
+        </collision>
     </link>
     <joint name="base_joint" type="fixed">
