Commit message: diff summer robot updated

File: diff_summer_robot_description/urdf/common_properties.xacro (robot description, xacro)
@@ -7,3 +7,30 @@
         <color rgba="0.5 0.5 0.5 1.0"/>
     </material>
+    <xacro:macro name="box_inertia" params="l w h m o_xyz o_rpy">
+        <inertial>
+                <origin xyz="${o_xyz}" rpy="${o_rpy}"/>
+                <mass value="${m}"/>
+                <inertia ixx="${m*(w*w+h*h)/12.0}" ixy="0.0" ixz="0.0"
+                         iyy="${m*(l*l+h*h)/12.0}" iyz="0.0"
+                         izz="${m*(w*w+l*l)/12.0}"/>
+        </inertial>
+    </xacro:macro>
+    <xacro:macro name="cylinder_inertia" params="r l m o_xyz o_rpy">
+        <inertial>
+                <origin xyz="${o_xyz}" rpy="${o_rpy}"/>
+                <mass value="${m}"/>
+                <inertia ixx="${m*(3*r*r+l*l)/12.0}" ixy="0.0" ixz="0.0"
+                         iyy="${m*(l*l+3*r*r)/12.0}" iyz="0.0"
+                         izz="${m*(r*r)/2.0}"/>
+        </inertial>
+    </xacro:macro>
+    <xacro:macro name="sphere_inertia" params="r m o_xyz o_rpy">
+        <inertial>
+                <origin xyz="${o_xyz}" rpy="${o_rpy}"/>
+                <mass value="${m}"/>
+                <inertia ixx="${2*m*r*r/5.0}" ixy="0.0" ixz="0.0"
+                         iyy="${2*m*r*r/5.0}" iyz="0.0"
+                         izz="${2*m*r*r/5.0}"/>
+        </inertial>
+    </xacro:macro>
 </robot>
