Commit message: Completed the mobile base to be compatible with gazebo. Still need to add the control

File: diff_summer_robot_description/urdf/mobile_base.xacro (robot description, xacro)
@@ -8,4 +8,5 @@
     <xacro:macro name="wheel_link" params="prefix">
         <link name="${prefix}_wheel_link">
+            <xacro:cylinder_inertia r="${wheel_radius}" l="${wheel_length}" m="1.0" o_xyz="0.0 0.0 0.0" o_rpy="${pi / 2.0} 0.0 0.0"/>
             <visual>
                 <origin xyz="0.0 0.0 0.0" rpy="${pi / 2.0} 0.0 0.0"/>
@@ -15,19 +16,33 @@
                 <material name="grey"/>
             </visual>
+            <collision>
+                <origin xyz="0.0 0.0 0.0" rpy="${pi / 2.0} 0.0 0.0"/>
+                <geometry>
+                    <sphere radius="${wheel_radius}"/>
+                </geometry>
+            </collision>
         </link>
     </xacro:macro>
     <link name="base_footprint"/>
     <link name="base_link">
+        <xacro:box_inertia l="${base_length}" w="${base_width}" h="${base_height}" m="5.0" o_xyz="0.0 0.0 ${base_height / 2.0}" o_rpy="0.0 0.0 0.0"/>
         <visual>
             <geometry>
                 <box size="${base_length} ${base_width} ${base_height}"/>
             </geometry>
-            <origin xyz="0.0 0.0 0.1" rpy="0.0 0.0 0.0"/>
+            <origin xyz="0.0 0.0 ${base_height / 2.0}" rpy="0.0 0.0 0.0"/>
             <material name="green"/>
         </visual>
+        <collision>
+            <origin xyz="0.0 0.0 ${base_height / 2.0}" rpy="0.0 0.0 0.0"/>
+            <geometry>
+                <box size="${base_length} ${base_width} ${base_height}"/>
+            </geometry>
+        </collision>
     </link>
     <xacro:wheel_link prefix="right"/>
     <xacro:wheel_link prefix="left"/>
     <link name="caster_wheel_link">
+        <xacro:sphere_inertia r="${wheel_radius / 2.0}" m="0.5" o_xyz="0.0 0.0 0.0" o_rpy="0.0 0.0 0.0"/>
         <visual>
             <origin xyz="0.0 0.0 0.0" rpy="0.0 0.0 0.0"/>
@@ -37,4 +52,10 @@
             <material name="grey"/>
         </visual>
+        <collision>
+            <origin xyz="0.0 0.0 0.0" rpy="0.0 0.0 0.0"/>
+            <geometry>
+                <sphere radius="${wheel_radius / 2.0}"/>
+            </geometry>
+        </collision>
     </link>
     <joint name="base_joint" type="fixed">
