Commit message: Completed movement in summer project tested lidar and camera in tutor

File: diff_summer_robot_description/urdf/diff_summer_robot.urdf.xacro (robot description, xacro)
@@ -3,3 +3,4 @@
     <xacro:include filename="$(find diff_summer_robot_description)/urdf/common_properties.xacro"/>
     <xacro:include filename="$(find diff_summer_robot_description)/urdf/mobile_base.xacro"/>
+    <xacro:include filename="$(find diff_summer_robot_description)/urdf/mobile_base_gazebo.xacro"/>
 </robot>

File: diff_summer_robot_description/urdf/tutor/common_properties_tutor.xacro (robot description, xacro)
@@ -6,4 +6,7 @@
     <material name="grey">
         <color rgba="0.5 0.5 0.5 1.0"/>
+    </material>
+    <material name="black">
+        <color rgba="0.05 0.05 0.05 1.0"/>
     </material>
     <xacro:macro name="box_inertia" params="m x y z o_xyz o_rpy">

File: diff_summer_robot_description/urdf/tutor/diff_summer_robot_tutor.urdf.xacro (robot description, xacro)
@@ -4,3 +4,5 @@
     <xacro:include filename="$(find diff_summer_robot_description)/urdf/tutor/mobile_base_tutor.xacro"/>
     <xacro:include filename="$(find diff_summer_robot_description)/urdf/tutor/mobile_base_gazebo_tutor.xacro"/>
+    <xacro:include filename="$(find diff_summer_robot_description)/urdf/tutor/camera_tutor.xacro"/>
+    <xacro:include filename="$(find diff_summer_robot_description)/urdf/tutor/lidar_tutor.xacro"/>
 </robot>
