Commit message: More closer to being able to simulate my custom ur

File: custom_ur_description/urdf/custom_ur.urdf.xacro (robot description, xacro)
@@ -5,7 +5,9 @@
    <!-- import main macro -->
    <xacro:include filename="$(find ur_description)/urdf/ur_macro.xacro"/>
+   <!-- Import macros -->
+   <xacro:include filename="$(find robotiq_description)/urdf/robotiq_2f_85_macro.urdf.xacro" />
    <!-- possible 'ur_type' values: ur3, ur3e, ur5, ur5e, ur10, ur10e, ur16e, ur20, ur30 -->
    <!-- the default value should raise an error in case this was called without defining the type -->
-   <xacro:arg name="ur_type" default="ur5x"/>
+   <xacro:arg name="ur_type" default="ur10e"/>
    <!-- parameters -->
    <xacro:arg name="tf_prefix" default="" />
@@ -40,5 +42,5 @@
    <xacro:arg name="tool_tcp_port" default="54321" />
      <!-- Simulation parameters -->
-   <xacro:arg name="use_fake_hardware" default="false" />
+   <xacro:arg name="use_fake_hardware" default="true" />
    <xacro:arg name="fake_sensor_commands" default="false" />
    <xacro:arg name="sim_gazebo" default="false" />
@@ -112,3 +114,6 @@
     </gazebo>
   </xacro:if>
+  <xacro:robotiq_gripper name="RobotiqGripperHardwareInterface" prefix="" parent="$(arg tf_prefix)tool0" use_fake_hardware="$(arg use_fake_hardware)">
+        <origin xyz="0 0 0" rpy="0 0 0" />
+  </xacro:robotiq_gripper>
 </robot>

Commit message: Added the pedestal to urdf

File: custom_ur_description/urdf/custom_ur.urdf.xacro (robot description, xacro)
@@ -8,4 +8,5 @@
    <!-- <xacro:include filename="$(find robotiq_description)/urdf/robotiq_2f_85_macro.urdf.xacro" /> -->
    <xacro:include filename="$(find custom_robotiq_description)/urdf/robotiq_2f85_macro.urdf.xacro" />
+   <xacro:include filename="$(find custom_robotiq_description)/urdf/robotiq_camera.xacro" />
    <!-- possible 'ur_type' values: ur3, ur3e, ur5, ur5e, ur10, ur10e, ur16e, ur20, ur30 -->
    <!-- the default value should raise an error in case this was called without defining the type -->
@@ -54,9 +55,44 @@
    <!-- create link fixed to the "world" -->
    <link name="world" />
+   <!-- pedestal -->
+   <xacro:property name="p_w" value="0.728"/>
+   <xacro:property name="p_d" value="0.752"/>
+   <xacro:property name="p_h" value="0.863"/>
+   <xacro:property name="p_m" value="37.1"/>
+   <link name="vention_pedestal">
+      <inertial>
+        <origin xyz="-379.5e-03 407.0e-03 -320.0e-03" rpy="${pi/2} 0.0 0.0"/>
+        <mass value="${p_m}"/>
+        <inertia ixx="${p_m*0.083333*(p_d*p_d + p_h*p_h)}" ixy="0.0" ixz="0.0" iyy="${p_m*0.083333*(p_w*p_w + p_h*p_h)}" iyz="0.0" izz="${p_m*0.083333*(p_w*p_w + p_d*p_d)}"/>
+      </inertial>
+      <visual>
+        <origin xyz="-379.5e-03 407.0e-03 -320.0e-03" rpy="${pi/2} 0.0 0.0"/>
+        <geometry>
+          <mesh filename="file://$(find custom_ur_description)/meshes/vention_pedestal.stl" scale="0.001 0.001 0.001"/>
+        </geometry>
+      </visual>
+      <collision>
+        <origin xyz="-379.5e-03 407.0e-03 -320.0e-03" rpy="${pi/2} 0.0 0.0"/>
+        <geometry>
+          <mesh filename="file://$(find custom_ur_description)/meshes/vention_pedestal.stl" scale="0.001 0.001 0.001"/>
+        </geometry>
+      </collision>
+   </link>
+   <joint name="world_pedestal_joint" type="fixed">
+    <parent link="world"/>
+    <child link="vention_pedestal"/>
+    <origin xyz="0.0 0.0 0.0" rpy="0.0 0.0 0.0"/>
+   </joint>
+   <!-- <joint name="pedestal_base_joint" type="fixed">
+    <parent link="vention_pedestal"/>
+    <child link="child_link"/>
+    <origin xyz="0.0 0.0 0.0" rpy="0.0 0.0 0.0"/>
+   </joint>
+    -->
    <!-- arm -->
    <xacro:ur_robot
      name="$(arg name)"
      tf_prefix="$(arg tf_prefix)"
-     parent="world"
+     parent="vention_pedestal"
      joint_limits_parameters_file="$(arg joint_limit_params)"
      kinematics_parameters_file="$(arg kinematics_params)"
@@ -92,5 +128,5 @@
      trajectory_port="$(arg trajectory_port)"
      >
-     <origin xyz="0 0 0" rpy="0 0 0" />          <!-- position robot in the world -->
+     <origin xyz="0 0 0.838" rpy="0 0 0" />          <!-- position robot in the world -->
    </xacro:ur_robot>
    <xacro:if value="$(arg sim_gazebo)">
@@ -123,4 +159,5 @@
         <origin xyz="0 0 0" rpy="0 0 0" />
   </xacro:robotiq_gripper> -->
-  <xacro:robotiq_gripper name="RobotiqGripperHardwareInterface" prefix="" parent="$(arg tf_prefix)tool0" bringup="$(arg sim_gazebo)"/>
+  <xacro:robotiq_camera prefix="$(arg tf_prefix)" parent="$(arg tf_prefix)tool0"/>
+  <xacro:robotiq_gripper name="RobotiqGripperHardwareInterface" prefix="" parent="robotiq_camera" bringup="$(arg sim_gazebo)" fixed="true"/>
 </robot>

Commit message: Added a camera to teh summer project

File: custom_ur_description/urdf/custom_ur.urdf.xacro (robot description, xacro)
@@ -19,5 +19,5 @@
    <xacro:arg name="physical_params" default="$(find ur_description)/config/$(arg ur_type)/physical_parameters.yaml"/>
    <xacro:arg name="visual_params" default="$(find ur_description)/config/$(arg ur_type)/visual_parameters.yaml"/>
-   <xacro:arg name="transmission_hw_interface" default=""/>
+   <!-- <xacro:arg name="transmission_hw_interface" default=""/> -->
    <xacro:arg name="safety_limits" default="false"/>
    <xacro:arg name="safety_pos_margin" default="0.15"/>
@@ -59,4 +59,32 @@
    <!-- pedestal -->
    <xacro:robot_stand parent="world" />
+   <!-- Not in jazzy remove from below entries -->
+    <!-- ###
+    transmission_hw_interface="$(arg transmission_hw_interface)"
+    use_fake_hardware="$(arg use_fake_hardware)"
+    fake_sensor_commands="$(arg fake_sensor_commands)"
+    sim_gazebo="$(arg sim_gazebo)"
+    sim_ignition="$(arg sim_ignition)"
+    headless_mode="$(arg headless_mode)"
+    initial_positions="${xacro.load_yaml(initial_positions_file)}"
+    use_tool_communication="$(arg use_tool_communication)"
+    tool_voltage="$(arg tool_voltage)"
+    tool_parity="$(arg tool_parity)"
+    tool_baud_rate="$(arg tool_baud_rate)"
+    tool_stop_bits="$(arg tool_stop_bits)"
+    tool_rx_idle_chars="$(arg tool_rx_idle_chars)"
+    tool_tx_idle_chars="$(arg tool_tx_idle_chars)"
+    tool_device_name="$(arg tool_device_name)"
+    tool_tcp_port="$(arg tool_tcp_port)"
+    robot_ip="$(arg robot_ip)"
+    script_filename="$(arg script_filename)"
+    output_recipe_filename="$(arg output_recipe_filename)"
+    input_recipe_filename="$(arg input_recipe_filename)"
+    reverse_ip="$(arg reverse_ip)"
+    script_command_port="$(arg script_command_port)"
+    reverse_port="$(arg reverse_port)"
+    script_sender_port="$(arg script_sender_port)"
+    trajectory_port="$(arg trajectory_port)"
+    ### -->
    <!-- arm -->
    <xacro:ur_robot
@@ -68,8 +96,8 @@
      physical_parameters_file="$(arg physical_params)"
      visual_parameters_file="$(arg visual_params)"
-     transmission_hw_interface="$(arg transmission_hw_interface)"
      safety_limits="$(arg safety_limits)"
      safety_pos_margin="$(arg safety_pos_margin)"
      safety_k_position="$(arg safety_k_position)"
+     transmission_hw_interface="$(arg transmission_hw_interface)"
      use_fake_hardware="$(arg use_fake_hardware)"
      fake_sensor_commands="$(arg fake_sensor_commands)"

File: diff_summer_robot_description/urdf/common_properties.xacro (robot description, xacro)
@@ -6,4 +6,7 @@
     <material name="grey">
         <color rgba="0.5 0.5 0.5 1.0"/>
+    </material>
+    <material name="black">
+        <color rgba="0.05 0.05 0.05 1.0"/>
     </material>
     <xacro:macro name="box_inertia" params="l w h m o_xyz o_rpy">

File: diff_summer_robot_description/urdf/diff_summer_robot.urdf.xacro (robot description, xacro)
@@ -4,3 +4,4 @@
     <xacro:include filename="$(find diff_summer_robot_description)/urdf/mobile_base.xacro"/>
     <xacro:include filename="$(find diff_summer_robot_description)/urdf/mobile_base_gazebo.xacro"/>
+    <xacro:include filename="$(find diff_summer_robot_description)/urdf/camera.xacro"/>
 </robot>
