Commit message: Implemented the qcar simulation in gazebo harmonic

File: qcar_description/urdf/qcar.gazebo.xacro (robot description, xacro)
@@ -1,211 +1,123 @@
 <?xml version="1.0"?>
 <robot name="QCar" xmlns:xacro="http://www.ros.org/wiki/xacro">
+  <xacro:property name="max_steering_angle" value="0.3"/>
+  <xacro:property name="axle_vel_limit" value="244.8696"/>
+  <link name="camera_rgb_optical_link"/>
+  <joint name="camera_rgb_optical_joint" type="fixed">
+    <!-- these values have to be these values otherwise the gazebo camera
+        image won't be aligned properly with the frame it is supposedly
+        originating from -->
+    <origin xyz="0.01 0 0" rpy="${-pi/2} 0 ${-pi/2}"/>
+    <parent link="camera_rgb"/>
+    <child link="camera_rgb_optical_link"/>
+  </joint>
 <!-- Define all the computer vision sernsor properties -->
 	<gazebo reference="camera_rgb">
     <!-- <material>Gazebo/Green</material> -->
     <sensor type="camera" name="intelrealsense_rgb">
-    	<pose>0 0 0 0 0 0</pose>
-    	<!-- <pose>0.081686 0.031547 0.15445 0 0 0</pose> -->
+      <always_on>1</always_on>
       <update_rate>60.0</update_rate>
+      <visualize>true</visualize>
+      <topic>qcar/rgb/image_raw</topic>
       <camera name="rgb">
         <horizontal_fov>1.21126</horizontal_fov>
         <image>
-          <width>640</width>
-          <height>480</height>
-          <format>R8G8B8</format>
+            <width>640</width>
+            <height>480</height>
+            <format>R8G8B8</format>
         </image>
         <clip>
-          <near>0.02</near>
-          <far>300</far>
+            <near>0.02</near>
+            <far>300</far>
         </clip>
+        <noise>
+            <type>gaussian</type>
+            <mean>0.0</mean>
+            <stddev>0.001</stddev>
+        </noise>
+        <distortion>
+          <k1>0.0</k1>
+          <k2>0.0</k2>
+          <k3>0.0</k3>
+          <p1>0.0</p1>
+          <p2>0.0</p2>
+        </distortion>
+        <optical_frame_id>camera_rgb_optical_link</optical_frame_id>
+        <camera_info_topic>qcar/rgb/camera_info</camera_info_topic>
       </camera>
-      <plugin name="camera_controller" filename="libgazebo_ros_camera.so">
-        <alwaysOn>true</alwaysOn>
-        <updateRate>0.0</updateRate>
-        <cameraName>qcar/rgb</cameraName>
-        <imageTopicName>image_color</imageTopicName>
-        <cameraInfoTopicName>camera_info</cameraInfoTopicName>
-        <frameName>camera_rgb</frameName>
-        <hackBaseline>0.07</hackBaseline>
-        <distortionK1>0.0</distortionK1>
-        <distortionK2>0.0</distortionK2>
-        <distortionK3>0.0</distortionK3>
-        <distortionT1>0.0</distortionT1>
-        <distortionT2>0.0</distortionT2>
-      </plugin>
     </sensor>
   </gazebo>
-  <gazebo reference="camera_csi_front">
-    <!-- <material>Gazebo/Green</material> -->
-    <sensor type="camera" name="csi_front">
-    	<pose>0 0 0 0 0 0</pose>
-    	<!-- <pose>0.081686 0.031547 0.15445 0 0 0</pose> -->
-      <update_rate>60.0</update_rate>
-      <camera name="front">
-        <horizontal_fov>2.79253</horizontal_fov>
-        <image>
-          <width>1280</width>
-          <height>640</height>
-          <format>R8G8B8</format>
-        </image>
-        <clip>
-          <near>0.02</near>
-          <far>300</far>
-        </clip>
-      </camera>
-      <plugin name="camera_controller" filename="libgazebo_ros_camera.so">
-        <alwaysOn>true</alwaysOn>
-        <updateRate>0.0</updateRate>
-        <cameraName>qcar/csi_front</cameraName>
-        <imageTopicName>image_raw</imageTopicName>
-        <cameraInfoTopicName>camera_info</cameraInfoTopicName>
-        <frameName>camera_csi_front</frameName>
-        <hackBaseline>0.07</hackBaseline>
-        <distortionK1>-0.264598808</distortionK1>
-        <distortionK2>0.0156281135</distortionK2>
-        <distortionK3>0.0822019378</distortionK3>
-        <distortionT1>0.0000652954</distortionT1>
-        <distortionT2>0.0053984313</distortionT2>
-      </plugin>
-    </sensor>
-  </gazebo>
-  <gazebo reference="camera_csi_right">
-    <!-- <material>Gazebo/Green</material> -->
-    <sensor type="camera" name="csi_right">
-    	<pose>0 0 0 0 0 0</pose>
-    	<!-- <pose>0.081686 0.031547 0.15445 0 0 0</pose> -->
-      <update_rate>60.0</update_rate>
-      <camera name="right">
-        <horizontal_fov>2.79253</horizontal_fov>
-        <image>
-          <width>1280</width>
-          <height>640</height>
-          <format>R8G8B8</format>
-        </image>
-        <clip>
-          <near>0.02</near>
-          <far>300</far>
-        </clip>
-      </camera>
-      <plugin name="camera_controller" filename="libgazebo_ros_camera.so">
-        <alwaysOn>true</alwaysOn>
-        <updateRate>0.0</updateRate>
-        <cameraName>qcar/csi_right</cameraName>
-        <imageTopicName>image_raw</imageTopicName>
-        <cameraInfoTopicName>camera_info</cameraInfoTopicName>
-        <frameName>camera_csi_right</frameName>
-        <hackBaseline>0.07</hackBaseline>
-       	<distortionK1>-0.264598808</distortionK1>
-        <distortionK2>0.0156281135</distortionK2>
-        <distortionK3>0.0822019378</distortionK3>
-        <distortionT1>0.0000652954</distortionT1>
-        <distortionT2>0.0053984313</distortionT2>
-      </plugin>
-    </sensor>
-  </gazebo>
-  <gazebo reference="camera_csi_back">
-    <!-- <material>Gazebo/Green</material> -->
-    <sensor type="camera" name="csi_back">
-    	<pose>0 0 0 0 0 0</pose>
-    	<!-- <pose>0.081686 0.031547 0.15445 0 0 0</pose> -->
-      <update_rate>60.0</update_rate>
-      <camera name="back">
-        <horizontal_fov>2.79253</horizontal_fov>
-        <image>
-          <width>1280</width>
-          <height>640</height>
-          <format>R8G8B8</format>
-        </image>
-        <clip>
-          <near>0.02</near>
-          <far>300</far>
-        </clip>
-      </camera>
-      <plugin name="camera_controller" filename="libgazebo_ros_camera.so">
-        <alwaysOn>true</alwaysOn>
-        <updateRate>0.0</updateRate>
-        <cameraName>qcar/csi_back</cameraName>
-        <imageTopicName>image_raw</imageTopicName>
-        <cameraInfoTopicName>camera_info</cameraInfoTopicName>
-        <frameName>camera_csi_back</frameName>
-        <hackBaseline>0.07</hackBaseline>
-        <distortionK1>-0.264598808</distortionK1>
-        <distortionK2>0.0156281135</distortionK2>
-        <distortionK3>0.0822019378</distortionK3>
-        <distortionT1>0.0000652954</distortionT1>
-        <distortionT2>0.0053984313</distortionT2>
-      </plugin>
-    </sensor>
-  </gazebo>
-  <gazebo reference="camera_csi_left">
-    <!-- <material>Gazebo/Green</material> -->
-    <sensor type="camera" name="csi_left">
-    	<pose>0 0 0 0 0 0</pose>
-    	<!-- <pose>0.081686 0.031547 0.15445 0 0 0</pose> -->
-      <update_rate>60.0</update_rate>
-      <camera name="left">
-        <horizontal_fov>2.79253</horizontal_fov>
-        <image>
-          <width>1280</width>
-          <height>640</height>
-          <format>R8G8B8</format>
-        </image>
-        <clip>
-          <near>0.02</near>
-          <far>300</far>
-        </clip>
-      </camera>
-      <plugin name="camera_controller" filename="libgazebo_ros_camera.so">
-        <alwaysOn>true</alwaysOn>
-        <updateRate>0.0</updateRate>
-        <cameraName>qcar/csi_left</cameraName>
-        <imageTopicName>image_raw</imageTopicName>
-        <cameraInfoTopicName>camera_info</cameraInfoTopicName>
-        <frameName>camera_csi_left</frameName>
-        <hackBaseline>0.07</hackBaseline>
-        <distortionK1>-0.264598808</distortionK1>
-        <distortionK2>0.0156281135</distortionK2>
-        <distortionK3>0.0822019378</distortionK3>
-        <distortionT1>0.0000652954</distortionT1>
-        <distortionT2>0.0053984313</distortionT2>
-      </plugin>
-    </sensor>
-  </gazebo>
-  <gazebo reference="lidar">
-    <sensor type="ray" name="head_rplidar_sensor">
-      <pose>0 0 0.010 -0 0</pose>
-      <visualize>true</visualize>
-      <!-- <visualize>false</visualize> -->
-      <alwaysOn>true</alwaysOn>
-      <update_rate>30</update_rate>
-      <ray>
-        <scan>
-          <horizontal>
-            <samples>240</samples>
-            <resolution>1</resolution>
-            <min_angle>-3.14159</min_angle>
-            <max_angle>3.14159</max_angle>
-          </horizontal>
-        </scan>
-        <range>
-          <min>0.10</min>
-          <max>12.0</max>
-          <resolution>0.01</resolution>
-        </range>
-        <noise>
-          <type>gaussian</type>
-          <!-- Noise parameters based on published spec for Hokuyo laser
-               achieving "+-30mm" accuracy at range < 10m.  A mean of 0.0m and
-               stddev of 0.01m will put 99.7% of samples within 0.03m of the true
-               reading. -->
-          <mean>0.0</mean>
-          <stddev>0.01</stddev>
-        </noise>
-      </ray>
-      <plugin name="gazebo_ros_head_rplidar_controller" filename="libgazebo_ros_laser.so">
-        <topicName>/qcar/lidar</topicName>
-        <frameName>lidar</frameName>
-      </plugin>
-    </sensor>
+  <!-- Gazebo Control -->
+  <ros2_control name="control" type="system">
+    <hardware>
+      <plugin>gz_ros2_control/GazeboSimSystem</plugin>
+    </hardware>
+    <joint name="left_steering_joint">
+      <command_interface name="position">
+        <param name="min">${-max_steering_angle}</param>
+        <param name="max">${max_steering_angle}</param>
+      </command_interface>
+      <state_interface name="position"/>
+      <state_interface name="velocity"/>
+      <state_interface name="effort"/>
+    </joint>
+    <joint name="right_steering_joint">
+      <param name="mimic">left_steering_joint</param> <!-- Command this joint -->
+      <param name="multiplier">1</param> <!-- Move in the opposite direction -->
+      <state_interface name="position"/>
+      <state_interface name="velocity"/>
+      <state_interface name="effort"/>
+    </joint>
+    <joint name="right_front_axle">
+      <command_interface name="velocity">
+        <param name="min">${-axle_vel_limit}</param>
+        <param name="max">${axle_vel_limit}</param>
+      </command_interface>
+      <state_interface name="position"/>
+      <state_interface name="velocity"/>
+      <state_interface name="effort"/>
+    </joint>
+    <joint name="left_front_axle">
+      <param name="mimic">right_front_axle</param> <!-- Command this joint -->
+      <param name="multiplier">-1</param> <!-- Move in the opposite direction -->
+      <state_interface name="position"/>
+      <state_interface name="velocity"/>
+      <state_interface name="effort"/>
+    </joint>
+    <joint name="right_rear_axle">
+      <command_interface name="velocity">
+        <param name="min">${-axle_vel_limit}</param>
+        <param name="max">${axle_vel_limit}</param>
+      </command_interface>
+      <state_interface name="position"/>
+      <state_interface name="velocity"/>
+      <state_interface name="effort"/>
+    </joint>
+    <joint name="left_rear_axle">
+      <command_interface name="velocity">
+        <param name="min">${-axle_vel_limit}</param>
+        <param name="max">${axle_vel_limit}</param>
+      </command_interface>
+      <state_interface name="position"/>
+      <state_interface name="velocity"/>
+      <state_interface name="effort"/>
+    </joint>
+  </ros2_control>
+  <gazebo>
+    <plugin filename="gz-sim-joint-state-publisher-system" name="gz::sim::systems::JointStatePublisher">
+      <topic>joint_states</topic>
+      <joint_name>left_steering_joint</joint_name>
+      <joint_name>right_steering_joint</joint_name>
+      <joint_name>left_front_axle</joint_name>
+      <joint_name>right_front_axle</joint_name>
+      <joint_name>left_rear_axle</joint_name>
+      <joint_name>right_rear_axle</joint_name>
+    </plugin>
+    <plugin filename="gz_ros2_control-system" name="gz_ros2_control::GazeboSimROS2ControlPlugin">
+      <parameters>$(find qcar_gazebo)/config/gz_ros2_control.yaml</parameters>
+    </plugin>
+    <plugin filename="gz-sim-sensors-system" name="gz::sim::systems::Sensors">
+        <render_engine>ogre2</render_engine>
+    </plugin>
   </gazebo>
 </robot>

File: qcar_description/urdf/qcar.materials.xacro (robot description, xacro)
@@ -2,5 +2,5 @@
 <robot name="QCar" xmlns:xacro="http://www.ros.org/wiki/xacro">
 	<material name="black">
-    <color rgba="0.0 0.0 0.0 1.0"/>
+    <color rgba="0.1 0.1 0.1 1.0"/>
   </material>
   <material name="blue">
@@ -11,5 +11,5 @@
   </material>
   <material name="grey">
-    <color rgba="0.2 0.2 0.2 1.0"/>
+    <color rgba="0.5 0.5 0.5 1.0"/>
   </material>
   <material name="orange">

File: qcar_description/urdf/qcar_ros2.urdf.xacro (robot description, xacro)
@@ -31,5 +31,5 @@
   <xacro:macro name="QCar" params="parent prefix *origin">
     <!-- includes -->
-    <xacro:include filename="$(find qcar_description)/urdf/qcar.gazebo.xacro" />
+    <!-- <xacro:include filename="$(find qcar_description)/urdf/qcar.gazebo.xacro" /> -->
     <xacro:include filename="$(find qcar_description)/urdf/qcar.materials.xacro" />
     <!-- Degree-to-radian conversions -->
@@ -126,9 +126,9 @@
     <!-- base_link must have geometry so that its axes can be displayed in
          rviz. -->
-    <joint name="$base_joint" type="fixed">
+    <!-- <joint name="$base_joint" type="fixed">
       <xacro:insert_block name="origin" />
       <parent link="${parent}"/>
       <child link="${prefix}base_link" />
-    </joint>
+    </joint> -->
    <link name="base_link" />
     <!-- Chassis -->
@@ -139,7 +139,8 @@
         <geometry>
     <!-- <box size="${chassis_length} ${chassis_width} ${chassis_height}"/> -->
-    <mesh filename="file://$(find qcar_description)/meshes/QCarBody.stl" scale="0.001 0.001 0.001"/>
+          <mesh filename="file://$(find qcar_description)/meshes/QCarBody.stl" scale="0.001 0.001 0.001"/>
         </geometry>
         <!-- <material name="chassis_mat"/> -->
+        <material name="grey"/>
       </visual>
       <collision>
@@ -148,10 +149,10 @@
         <geometry>
     <!-- <box size="${chassis_length} ${chassis_width} ${chassis_height}"/> -->
-    <mesh filename="file://$(find qcar_description)/meshes/QCarBody.stl" scale="0.001 0.001 0.001"/>
+          <mesh filename="file://$(find qcar_description)/meshes/QCarBody.stl" scale="0.001 0.001 0.001"/>
         </geometry>
       </collision>
       <xacro:solid_cuboid_inertial
-    width="${chassis_length}" depth="${chassis_width}"
-    height="${chassis_height}" mass="${chassis_mass}">
+                                  width="${chassis_length}" depth="${chassis_width}"
+                                  height="${chassis_height}" mass="${chassis_mass}">
         <origin xyz="0 0 0"/>
       </xacro:solid_cuboid_inertial>
@@ -220,5 +221,6 @@
         <!-- <origin xyz=".2 0 0" rpy="0 0 0"/> -->
         <!-- ___________________xyz is wrong, need to update_______________________________ -->
-        <origin rpy="0 0 -1.5708" xyz="0.12887 -0.06755 0.093029"/>
+        <!-- <origin rpy="0 0 -1.5708" xyz="0.12887 -0.06755 0.093029"/> -->
+        <origin rpy="0 0 -1.5708" xyz="0.012887 -0.06755 0.093029"/>
         <!-- <origin rpy="0 0 0" xyz="0 0 0"/> -->
         <parent link="base"/>
@@ -239,5 +241,6 @@
         <!-- <origin xyz=".2 0 0" rpy="0 0 0"/> -->
         <!-- ___________________xyz is wrong, need to update_______________________________ -->
-        <origin rpy="0 0 1.5708" xyz="0.12784 0.052497 0.093029"/>
+        <!-- <origin rpy="0 0 1.5708" xyz="0.12784 0.052497 0.093029"/> -->
+         <origin rpy="0 0 1.5708" xyz="0.012784 0.052497 0.093029"/>
         <!-- <origin rpy="0 0 0" xyz="0 0 0"/> -->
         <parent link="base"/>
@@ -282,18 +285,20 @@
       <child link="left_front_axle_carrier"/>
       <axis xyz = "0 0 1"/>
-      <limit lower="-0.523599" upper="0.523599" effort="0.5649" velocity="4.553"/>
+      <!-- <limit lower="-0.523599" upper="0.523599" effort="0.5649" velocity="4.553"/> -->
+      <limit lower="-0.3" upper="0.3" effort="0.5649" velocity="4.553"/>
     </joint>
     <link name="left_front_axle_carrier">
       <xacro:null_inertial/>
     </link>
-    <joint name="left_front_axle" type="fixed">
+    <joint name="left_front_axle" type="continuous">
       <parent link="left_front_axle_carrier"/>
       <child link="left_front_wheel"/>
-      <axis xyz="0 0 1"/>
+      <axis xyz="0 1 0"/>
       <origin rpy="0 0 3.14159"/>
       <limit effort="5.12766" velocity="244.8696"/>
       <dynamics damping="0.1" friction="0.1"/>
-    </joint>
-    <!-- <transmission name="left_front_axle_trans">
+      <mimic joint="right_front_axle" multiplier="-1.0" offset="0"/>
+    </joint>
+    <transmission name="left_front_axle_trans">
       <type>transmission_interface/SimpleTransmission</type>
       <joint name="left_front_axle">
@@ -303,12 +308,12 @@
         <mechanicalReduction>1</mechanicalReduction>
       </actuator>
-    </transmission> -->
+    </transmission>
     <link name="left_front_wheel">
       <visual>
         <origin rpy="0 0 0" xyz="0 0 0"/>
         <geometry>
-    <mesh filename="file://$(find qcar_description)/meshes/QCarWheel.stl" scale="0.001 0.001 0.001"/>
-        </geometry>
-        <material name="red"/>
+          <mesh filename="file://$(find qcar_description)/meshes/QCarWheel.stl" scale="0.001 0.001 0.001"/>
+        </geometry>
+        <material name="black"/>
       </visual>
       <collision>
@@ -322,5 +327,5 @@
       height="${tire_width}" mass="${wheel_mass}"/>
     </link>
-    <!-- <transmission name="left_steering_trans">
+    <transmission name="left_steering_trans">
       <type>transmission_interface/SimpleTransmission</type>
       <joint name="left_steering_joint">
@@ -330,5 +335,5 @@
         <mechanicalReduction>1</mechanicalReduction>
       </actuator>
-    </transmission> -->
+    </transmission>
   <!-- ___base_link - > right_front_position_joint (fixed) -> right_steering_link -> right_steering_joint(revolote) -> right_front_axle_carrier -> right_front_axle(joint) (continuous) -> right_front_wheel_______________ -->
     <link name="right_front_axle_carrier">
@@ -342,5 +347,5 @@
       <dynamics damping="0.1" friction="0.1"/>
     </joint>
-    <!-- <transmission name="right_front_axle_trans">
+    <transmission name="right_front_axle_trans">
       <type>transmission_interface/SimpleTransmission</type>
       <joint name="right_front_axle">
@@ -350,5 +355,5 @@
         <mechanicalReduction>1</mechanicalReduction>
       </actuator>
-    </transmission> -->
+    </transmission>
     <link name="right_front_wheel">
       <visual>
@@ -357,5 +362,5 @@
     <mesh filename="file://$(find qcar_description)/meshes/QCarWheel.stl" scale="0.001 0.001 0.001"/>
         </geometry>
-        <material name="red"/>
+        <material name="black"/>
       </visual>
       <collision>
@@ -390,11 +395,13 @@
       </collision>
     </link>
-    <joint name="right_steering_joint" type="fixed">
+    <joint name="right_steering_joint" type="revolute">
       <parent link="right_steering_link"/>
       <child link="right_front_axle_carrier"/>
       <axis xyz = "0 0 1"/>
-      <limit lower="0.523599" upper="0.523599" effort="0.5649" velocity="4.553"/>
-    </joint>
-    <!-- <transmission name="right_steering_trans">
+      <!-- <limit lower="0.523599" upper="0.523599" effort="0.5649" velocity="4.553"/> -->
+      <limit lower="-0.3" upper="0.3" effort="0.5649" velocity="4.553"/>
+      <mimic joint="left_steering_joint" multiplier="1.0" offset="0"/>
+    </joint>
+    <transmission name="right_steering_trans">
       <type>transmission_interface/SimpleTransmission</type>
       <joint name="right_steering_joint">
@@ -404,5 +411,5 @@
         <mechanicalReduction>1</mechanicalReduction>
       </actuator>
-    </transmission> -->
+    </transmission>
     <!-- The upper portion is for the front -->
     <!-- Now is for the rear which only has axles -->
@@ -419,5 +426,5 @@
       <dynamics damping="0.1" friction="0.1"/>
     </joint>
-    <!-- <transmission name="left_rear_axle_trans">
+    <transmission name="left_rear_axle_trans">
       <type>transmission_interface/SimpleTransmission</type>
       <joint name="left_rear_axle">
@@ -427,5 +434,5 @@
         <mechanicalReduction>1</mechanicalReduction>
       </actuator>
-    </transmission> -->
+    </transmission>
     <link name="left_rear_wheel">
       <visual>
@@ -434,5 +441,5 @@
     <mesh filename="file://$(find qcar_description)/meshes/QCarWheel.stl" scale="0.001 0.001 0.001"/>
         </geometry>
-        <material name="red"/>
+        <material name="black"/>
       </visual>
       <collision>
@@ -462,5 +469,5 @@
       <dynamics damping="0.1" friction="0.1"/>
     </joint>
-    <!-- <transmission name="right_rear_axle_trans">
+    <transmission name="right_rear_axle_trans">
       <type>transmission_interface/SimpleTransmission</type>
       <joint name="right_rear_axle">
@@ -470,5 +477,5 @@
         <mechanicalReduction>1</mechanicalReduction>
       </actuator>
-    </transmission> -->
+    </transmission>
     <link name="right_rear_wheel">
       <visual>
@@ -477,5 +484,5 @@
     <mesh filename="file://$(find qcar_description)/meshes/QCarWheel.stl" scale="0.001 0.001 0.001"/>
         </geometry>
-        <material name="red"/>
+        <material name="black"/>
       </visual>
       <collision>
@@ -495,4 +502,25 @@
     </joint>
     <!-- The above is for the wheels and turning etc -->
+    <!-- Gazebo Parameters -->
+    <gazebo reference="base">
+      <mu1>0.0001</mu1>
+      <mu2>0.0001</mu2>
+    </gazebo>
+    <gazebo reference="right_front_wheel">
+      <mu1>100.0</mu1>
+      <mu2>100.0</mu2>
+    </gazebo>
+    <gazebo reference="left_front_wheel">
+      <mu1>100.0</mu1>
+      <mu2>100.0</mu2>
+    </gazebo>
+    <gazebo reference="right_rear_wheel">
+      <mu1>100.0</mu1>
+      <mu2>100.0</mu2>
+    </gazebo>
+    <gazebo reference="left_rear_wheel">
+      <mu1>100.0</mu1>
+      <mu2>100.0</mu2>
+    </gazebo>
     <!--<gazebo>
       <plugin name="gazebo_ros_control" filename="libgazebo_ros_control.so" />

File: qcar_description/urdf/qcar_system.urdf.xacro (robot description, xacro)
@@ -10,12 +10,12 @@
   <xacro:include filename="$(find qcar_description)/urdf/qcar.gazebo.xacro" />
   <!-- Import Rviz colors -->
-  <!--<xacro:include filename="$(find qcar_description)/gazebo/qcar.materials.xacro" />-->
+  <!-- <xacro:include filename="$(find qcar_description)/urdf/qcar.materials.xacro" /> -->
   <!-- Import diffbot ros2_control description -->
   <!-- <xacro:include filename="$(find qcar_description)/ros2_control/qcar_system.ros2_control.xacro" /> -->
   <!-- Used for fixing robot -->
-  <link name="world"/>
-  <gazebo reference="world">
-    <static>true</static>
-  </gazebo>
+  <!-- <link name="world"/> -->
+  <!-- <gazebo reference="world">
+    <static>false</static>
+  </gazebo> -->
   <xacro:QCar parent="world" prefix="$(arg prefix)">
     <origin xyz="0 0 0" rpy="0 0 0" />
